File: gsvesc_drv.sch (KiCad schematic (older format))
At the start: 38 parts

Commit message: aufräumen
Parts:
- U?: symbol gsvec:DRV8301DCAR -> gsvesc-rescue:DRV8301DCAR-gsvec
- U?: symbol gsvec:IRU1010-33 -> gsvesc-rescue:IRU1010-33-gsvec
Changed lines of the file:
@@
 DRV8301 / 5V Buck Converter
 $Comp
-L gsvec:DRV8301DCAR U?
+L gsvesc-rescue:DRV8301DCAR-gsvec U?
 U 1 1 5BF0D51D
 P 3650 2150
@@
 SH_C
 $Comp
-L gsvec:IRU1010-33 U?
+L gsvesc-rescue:IRU1010-33-gsvec U?
 U 1 1 5BFDC9B0
 P 2750 6600
