File: gsvesc_drv.sch (KiCad schematic (older format))
At the start: 38 parts

Commit message: Aufgeräumt Teil 2
Parts:
- U?: symbol gsvec:DRV8301DCAR -> gsvesc:DRV8301DCAR
- U?: symbol gsvec:IRU1010-33 -> gsvesc:IRU1010-33
Changed lines of the file:
@@
 DRV8301 / 5V Buck Converter
 $Comp
-L gsvec:DRV8301DCAR U?
+L gsvesc:DRV8301DCAR U?
 U 1 1 5BF0D51D
 P 3650 2150
+AR Path="/5BF0D51D" Ref="U?"  Part="1"
+AR Path="/5BECFAA4/5BF0D51D" Ref="U?"  Part="1"
 F 0 "U?" H 5050 2537 60  0000 C CNN
 F 1 "DRV8301DCAR" H 5050 2431 60  0000 C CNN
@@
 SH_C
 $Comp
-L gsvec:IRU1010-33 U?
+L gsvesc:IRU1010-33 U?
 U 1 1 5BFDC9B0
 P 2750 6600

Commit message: SCM Fertig
Parts:
- removed C? (x2): 100u, symbol Device:C
- added C24, C34: 100u/16V, Capacitor_SMD:CP_Elec_16x17.5, symbol Device:CP
- C14, C15, C18, C19, C21, C23, C33: renamed from C?; value 10u0 -> 10u0/16V; footprint (none) -> Capacitor_SMD:C_0805_2012Metric
- C16, C17, C20, C22, C25, C27, C28, C29, C30, C31: renamed from C?; footprint (none) -> Capacitor_SMD:C_0805_2012Metric
- C26, C32: renamed from C?; value 47u / 100V -> 47u0/100V; footprint (none) -> Capacitor_SMD:C_1210_3225Metric
- D4: renamed from D?; value B360-SMA -> B360_SMA; footprint (none) -> Diode_SMD:D_SMA
- L1: renamed from L?; footprint (none) -> Inductor_SMD:L_Bourns_SRN6045TA
- R12, R13, R14, R15, R16, R17, R18, R19, R20, R21, R22, R23, R24: renamed from R?; footprint (none) -> Resistor_SMD:R_0805_2012Metric
- U2: renamed from U?; footprint (none) -> Package_TO_SOT_SMD:SOT-223
- U3: renamed from U?; footprint DCA56_6P35X3P61 -> gsvesc:DRV8301DCAR
Connections:
- net +5V: now also C34.1
- net GND: now also C24.2, C34.2; no longer U2.4 (PAD_OUT)
- net VCC: now also C24.1

Commit message: design finished gerber created
Parts:
- removed C14: 10u0/16V, Capacitor_SMD:C_0805_2012Metric, symbol Device:C
- removed C24: 100u/16V, Capacitor_SMD:CP_Elec_16x17.5, symbol Device:CP
- C29, C30, C31: footprint Capacitor_SMD:C_0805_2012Metric -> Capacitor_SMD:C_0603_1608Metric
- C34: footprint Capacitor_SMD:CP_Elec_16x17.5 -> Capacitor_Tantalum_SMD:CP_EIA-3216-18_Kemet-A
Connections:
- net VCC: now also U2.4 (PAD_OUT)
- net SENSE_SUPPLY renamed SENSE_VBAT
- no-connect marks 0 -> 6
Other:
- moved on the sheet: U2
Changed lines of the file:
@@
 SL_C
 Text HLabel 9100 4000 0    50   Input ~ 0
-SENSE_SUPPLY
+SENSE_VBAT
 Text HLabel 9100 4550 0    50   Input ~ 0
 SENS_A
@@
 F 0 "C31" V 6900 4150 50  0000 C CNN
 F 1 "220n" V 7000 4200 50  0000 C CNN
-F 2 "Capacitor_SMD:C_0805_2012Metric" H 7088 3900 50  0001 C CNN
+F 2 "Capacitor_SMD:C_0603_1608Metric" H 7088 3900 50  0001 C CNN
 F 3 "~" H 7050 4050 50  0001 C CNN
 	1    7050 4050
@@
 F 0 "C30" V 6950 3650 50  0000 C CNN
 F 1 "220n" V 7000 3700 50  0000 C CNN
-F 2 "Capacitor_SMD:C_0805_2012Metric" H 7088 3400 50  0001 C CNN
+F 2 "Capacitor_SMD:C_0603_1608Metric" H 7088 3400 50  0001 C CNN
 F 3 "~" H 7050 3550 50  0001 C CNN
 	1    7050 3550
@@
 F 0 "C29" V 6900 3150 50  0000 C CNN
 F 1 "220n" V 7000 3200 50  0000 C CNN
-F 2 "Capacitor_SMD:C_0805_2012Metric" H 7088 2900 50  0001 C CNN
+F 2 "Capacitor_SMD:C_0603_1608Metric" H 7088 2900 50  0001 C CNN
 F 3 "~" H 7050 3050 50  0001 C CNN
 	1    7050 3050
@@
 L gsvesc:IRU1010-33 U2
 U 1 1 5BFDC9B0
-P 2750 6600
-F 0 "U2" H 2600 6700 50  0000 C CNN
-F 1 "IRU1010-33" H 2800 6600 50  0000 C CNN
-F 2 "Package_TO_SOT_SMD:SOT-223" H 2750 6600 50  0001 C CNN
-F 3 "" H 2750 6600 50  0001 C CNN
-	1    2750 6600
+P 2750 6500
+F 0 "U2" H 2600 6600 50  0000 C CNN
+F 1 "IRU1010-33" H 2800 6500 50  0000 C CNN
+F 2 "Package_TO_SOT_SMD:SOT-223" H 2750 6500 50  0001 C CNN
+F 3 "" H 2750 6500 50  0001 C CNN
+	1    2750 6500
 	1    0    0    -1
 $EndComp
@@
 $EndComp
 $Comp
-L Device:C C14
-U 1 1 5BFE26F3
-P 1700 6900
-F 0 "C14" H 1750 7000 50  0000 L CNN
-F 1 "10u0/16V" H 1700 6800 50  0000 L CNN
-F 2 "Capacitor_SMD:C_0805_2012Metric" H 1738 6750 50  0001 C CNN
-F 3 "~" H 1700 6900 50  0001 C CNN
-	1    1700 6900
-	1    0    0    -1
-$EndComp
-$Comp
 L Device:C C16
 U 1 1 5BFE2759
@@
 Wire Wire Line
 	4150 6750 4750 6750
-Wire Wire Line
-	1450 6750 1700 6750
-Connection ~ 1700 6750
-Wire Wire Line
-	1700 6750 2150 6750
 Connection ~ 2150 6750
 Wire Wire Line
@@
 	1700 7050 2150 7050
 Connection ~ 2150 7050
-Wire Wire Line
-	2150 7050 2750 7050
-Connection ~ 2750 7050
-Wire Wire Line
-	2750 7050 3350 7050
-Connection ~ 3350 7050
 Connection ~ 4150 7050
 Wire Wire Line
@@
 F 0 "C34" H 8668 2946 50  0000 L CNN
 F 1 "100u/16V" H 8668 2855 50  0000 L CNN
-F 2 "Capacitor_SMD:CP_Elec_16x17.5" H 8588 2750 50  0001 C CNN
+F 2 "Capacitor_Tantalum_SMD:CP_EIA-3216-18_Kemet-A" H 8588 2750 50  0001 C CNN
 F 3 "~" H 8550 2900 50  0001 C CNN
 	1    8550 2900
@@
 Connection ~ 8550 2750
 Connection ~ 8550 3050
-Wire Wire Line
-	3350 6750 3750 6750
-Wire Wire Line
-	3350 7050 3750 7050
-$Comp
-L Device:CP C24
-U 1 1 5C10EC7A
-P 3750 6900
-F 0 "C24" H 3800 7000 50  0000 L CNN
-F 1 "100u/16V" H 3750 6800 50  0000 L CNN
-F 2 "Capacitor_SMD:CP_Elec_16x17.5" H 3788 6750 50  0001 C CNN
-F 3 "~" H 3750 6900 50  0001 C CNN
-	1    3750 6900
-	1    0    0    -1
-$EndComp
-Connection ~ 3750 6750
-Wire Wire Line
-	3750 6750 4150 6750
-Connection ~ 3750 7050
-Wire Wire Line
-	3750 7050 4150 7050
+Connection ~ 3350 7050
+$Comp
+L power:PWR_FLAG #FLG0101
+U 1 1 5C11889B
+P 4150 6750
+F 0 "#FLG0101" H 4150 6825 50  0001 C CNN
+F 1 "PWR_FLAG" H 4150 6924 50  0000 C CNN
+F 2 "" H 4150 6750 50  0001 C CNN
+F 3 "~" H 4150 6750 50  0001 C CNN
+	1    4150 6750
+	1    0    0    -1
+$EndComp
+Wire Wire Line
+	1450 6750 2150 6750
+Wire Wire Line
+	3350 6750 3600 6750
+Wire Wire Line
+	2450 6750 2450 6650
+Wire Wire Line
+	2150 7050 2750 7050
+Wire Wire Line
+	3350 7050 4150 7050
+Wire Wire Line
+	2750 6950 2750 7050
+Connection ~ 2750 7050
+Wire Wire Line
+	2750 7050 3350 7050
+Wire Wire Line
+	3050 6650 3050 6750
+Wire Wire Line
+	3500 6950 3600 6950
+Wire Wire Line
+	3600 6950 3600 6750
+Connection ~ 3600 6750
+Wire Wire Line
+	3600 6750 4150 6750
+NoConn ~ 6450 2350
+NoConn ~ 3650 2450
+NoConn ~ 3650 2550
+NoConn ~ 3650 3250
+NoConn ~ 3650 4550
+NoConn ~ 3650 4650
 $EndSCHEMATC

Commit message: change inverter to npn :)
Parts:
- U2: symbol gsvesc:IRU1010-33 -> gsvesc-rescue:IRU1010-33-gsvesc
- U3: symbol gsvesc:DRV8301DCAR -> gsvesc-rescue:DRV8301DCAR-gsvesc
Changed lines of the file:
@@
 DRV8301 / 5V Buck Converter
 $Comp
-L gsvesc:DRV8301DCAR U?
+L gsvesc-rescue:DRV8301DCAR-gsvesc U?
 U 1 1 5BF0D51D
 P 3650 2150
@@
 SH_C
 $Comp
-L gsvesc:IRU1010-33 U2
+L gsvesc-rescue:IRU1010-33-gsvesc U2
 U 1 1 5BFDC9B0
 P 2750 6500

Commit message: test
Parts:
- added R38: 100k, Resistor_SMD:R_0805_2012Metric, symbol Device:R
- added R39: 3k2, Resistor_SMD:R_0805_2012Metric, symbol Device:R
Connections:
- net GND: now also R39.2
- net VBAT: now also R38.1
- net at U3.55 (EN_BUCK): now also R38.2, R39.1
- no-connect marks 6 -> 5
Changed lines of the file:
@@
 Title "GSVESC - DC Motor Controler"
 Date "2018-11-11"
-Rev "2.0"
+Rev "3.0"
 Comp ""
 Comment1 ""
@@
 Wire Wire Line
 	3600 6750 4150 6750
-NoConn ~ 6450 2350
 NoConn ~ 3650 2450
 NoConn ~ 3650 2550
@@
 NoConn ~ 3650 4550
 NoConn ~ 3650 4650
+$Comp
+L Device:R R38
+U 1 1 5DF0BDAB
+P 6850 1100
+F 0 "R38" H 6920 1146 50  0000 L CNN
+F 1 "100k" H 6920 1055 50  0000 L CNN
+F 2 "Resistor_SMD:R_0805_2012Metric" V 6780 1100 50  0001 C CNN
+F 3 "~" H 6850 1100 50  0001 C CNN
+	1    6850 1100
+	1    0    0    -1
+$EndComp
+$Comp
+L Device:R R39
+U 1 1 5DF0C0DB
+P 6850 1550
+F 0 "R39" H 6920 1596 50  0000 L CNN
+F 1 "3k2" H 6920 1505 50  0000 L CNN
+F 2 "Resistor_SMD:R_0805_2012Metric" V 6780 1550 50  0001 C CNN
+F 3 "~" H 6850 1550 50  0001 C CNN
+	1    6850 1550
+	1    0    0    -1
+$EndComp
+Wire Wire Line
+	6850 1250 6850 1350
+Wire Wire Line
+	6550 2350 6450 2350
+Wire Wire Line
+	6850 1700 6850 1900
+Wire Wire Line
+	6550 1350 6850 1350
+Wire Wire Line
+	6550 1350 6550 2350
+Connection ~ 6850 1350
+Wire Wire Line
+	6850 1350 6850 1400
+Text HLabel 6950 800  2    50   Input ~ 0
+VBAT
+Wire Wire Line
+	6850 950  6850 800
+Wire Wire Line
+	6850 800  6950 800
 $EndSCHEMATC

Commit message: gsesc v3, work in progress
Parts:
- added D5: D, Diode_SMD:D_SMA, symbol Device:D
- U2: symbol gsvesc-rescue:IRU1010-33-gsvesc -> gsvesc:IRU1010-33
- U3: symbol gsvesc-rescue:DRV8301DCAR-gsvesc -> gsvesc:DRV8301DCAR
Connections:
- net +5V: now also D5.1 (K)
- net GND: now also D5.2 (A)
Other:
- note added: "TVS 5V SMA"
Changed lines of the file:
@@
 $Descr A4 11693 8268
 encoding utf-8
-Sheet 3 6
-Title "GSVESC - DC Motor Controler"
+Sheet 3 5
+Title "GSESC - DC Motor Controler"
 Date "2018-11-11"
 Rev "3.0"
@@
 DRV8301 / 5V Buck Converter
 $Comp
-L gsvesc-rescue:DRV8301DCAR-gsvesc U?
+L gsvesc:DRV8301DCAR U?
 U 1 1 5BF0D51D
 P 3650 2150
@@
 SH_C
 $Comp
-L gsvesc-rescue:IRU1010-33-gsvesc U2
+L gsvesc:IRU1010-33 U2
 U 1 1 5BFDC9B0
 P 2750 6500
@@
 Wire Wire Line
 	6850 800  6950 800
+$Comp
+L Device:D D5
+U 1 1 5DF4B1D8
+P 9300 2900
+F 0 "D5" V 9254 2979 50  0000 L CNN
+F 1 "D" V 9345 2979 50  0000 L CNN
+F 2 "Diode_SMD:D_SMA" H 9300 2900 50  0001 C CNN
+F 3 "~" H 9300 2900 50  0001 C CNN
+	1    9300 2900
+	0    1    1    0
+$EndComp
+Wire Wire Line
+	8550 2750 9300 2750
+Wire Wire Line
+	8550 3050 9300 3050
+Text Notes 9200 2700 0    50   ~ 0
+TVS 5V SMA
 $EndSCHEMATC

Commit message: Update
Parts:
- C26, C32: value 47u0/100V -> 10u0/75V
- D5: value D -> SMBJ6.0CA; footprint Diode_SMD:D_SMA -> Diode_SMD:D_SMB
Changed lines of the file:
@@
 P 6600 5200
 F 0 "C26" H 6715 5246 50  0000 L CNN
-F 1 "47u0/100V" H 6715 5155 50  0000 L CNN
+F 1 "10u0/75V" H 6715 5155 50  0000 L CNN
 F 2 "Capacitor_SMD:C_1210_3225Metric" H 6638 5050 50  0001 C CNN
 F 3 "~" H 6600 5200 50  0001 C CNN
@@
 P 7900 2150
 F 0 "C32" H 8015 2196 50  0000 L CNN
-F 1 "47u0/100V" H 8015 2105 50  0000 L CNN
+F 1 "10u0/75V" H 8015 2105 50  0000 L CNN
 F 2 "Capacitor_SMD:C_1210_3225Metric" H 7938 2000 50  0001 C CNN
 F 3 "~" H 7900 2150 50  0001 C CNN
@@
 P 9300 2900
 F 0 "D5" V 9254 2979 50  0000 L CNN
-F 1 "D" V 9345 2979 50  0000 L CNN
-F 2 "Diode_SMD:D_SMA" H 9300 2900 50  0001 C CNN
+F 1 "SMBJ6.0CA" V 9345 2979 50  0000 L CNN
+F 2 "Diode_SMD:D_SMB" H 9300 2900 50  0001 C CNN
 F 3 "~" H 9300 2900 50  0001 C CNN
 	1    9300 2900

Commit message: implement remarks/changes from Alex
Parts:
- C29, C30, C31: footprint Capacitor_SMD:C_0603_1608Metric -> Capacitor_SMD:C_0805_2012Metric
Changed lines of the file:
@@
 F 0 "C31" V 6900 4150 50  0000 C CNN
 F 1 "220n" V 7000 4200 50  0000 C CNN
-F 2 "Capacitor_SMD:C_0603_1608Metric" H 7088 3900 50  0001 C CNN
+F 2 "Capacitor_SMD:C_0805_2012Metric" H 7088 3900 50  0001 C CNN
 F 3 "~" H 7050 4050 50  0001 C CNN
 	1    7050 4050
@@
 F 0 "C30" V 6950 3650 50  0000 C CNN
 F 1 "220n" V 7000 3700 50  0000 C CNN
-F 2 "Capacitor_SMD:C_0603_1608Metric" H 7088 3400 50  0001 C CNN
+F 2 "Capacitor_SMD:C_0805_2012Metric" H 7088 3400 50  0001 C CNN
 F 3 "~" H 7050 3550 50  0001 C CNN
 	1    7050 3550
@@
 F 0 "C29" V 6900 3150 50  0000 C CNN
 F 1 "220n" V 7000 3200 50  0000 C CNN
-F 2 "Capacitor_SMD:C_0603_1608Metric" H 7088 2900 50  0001 C CNN
+F 2 "Capacitor_SMD:C_0805_2012Metric" H 7088 2900 50  0001 C CNN
 F 3 "~" H 7050 3050 50  0001 C CNN
 	1    7050 3050
