File: gsvesc_drv.sch (KiCad schematic (older format))
At the start: 39 parts, among them U2 IRU1010-33, U3 DRV8301DCAR

Commit message: V3 finish, JLC ready
Parts:
- C28: value 15n0 -> 22n0
- R39: value 3k2 -> 3k90
Other:
- note added: "Ven < 1,2V buck off\nVBat_min=31V\n"
Changed lines of the file:
@@
 P 6850 2100
 F 0 "C28" H 6965 2146 50  0000 L CNN
-F 1 "15n0" H 6965 2055 50  0000 L CNN
+F 1 "22n0" H 6965 2055 50  0000 L CNN
 F 2 "Capacitor_SMD:C_0805_2012Metric" H 6888 1950 50  0001 C CNN
 F 3 "~" H 6850 2100 50  0001 C CNN
@@
 P 6850 1550
 F 0 "R39" H 6920 1596 50  0000 L CNN
-F 1 "3k2" H 6920 1505 50  0000 L CNN
+F 1 "3k90" H 6920 1505 50  0000 L CNN
 F 2 "Resistor_SMD:R_0805_2012Metric" V 6780 1550 50  0001 C CNN
 F 3 "~" H 6850 1550 50  0001 C CNN
@@
 Text Notes 9200 2700 0    50   ~ 0
 TVS 5V SMA
+Text Notes 7000 1400 0    50   ~ 0
+Ven < 1,2V buck off\nVBat_min=31V\n
 $EndSCHEMATC
