File: gsvesc_pwrctrl.sch (KiCad schematic (older format))
At the start: 13 parts

Commit message: aufräumen
Parts:
- Q?: symbol gsvec:IRF7749 -> gsvesc-rescue:IRF7749-gsvec
- Q?: symbol gsvec:LT1910 -> gsvesc-rescue:LT1910-gsvec
Changed lines of the file:
@@
 $EndComp
 $Comp
-L gsvec:IRF7749 Q?
+L gsvesc-rescue:IRF7749-gsvec Q?
 U 1 1 5C03A4C1
 P 6300 1550
@@
 $EndComp
 $Comp
-L gsvec:LT1910 Q?
+L gsvesc-rescue:LT1910-gsvec Q?
 U 1 1 5C03A92E
 P 5150 2350
