File: _autosave-gsvesc.kicad_pcb (KiCad board)
At the start: 4 copper layers, 111 x 111 mm, 113 parts, among them J1 Conn_01x06, J10 PHASE_C, J11 PHASE_A, J12 NTC, J13 PHASE_B, J14 Conn_02x04_Odd_Even, J2 Conn_01x06, J3 Conn_01x06, J4 Conn_01x05, J5 Conn_01x03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

Commit message: test
Parts:
- added C45: 680u/63V, Capacitor_SMD:CP_Elec_16x17.5, F.Cu at (175.0, 47.2)
- added C46: 680u/63V, Capacitor_SMD:CP_Elec_16x17.5, F.Cu at (196.2, 47.2)
- moved J7 80.3 mm to (182.2, 61.8)
- moved J8 47.1 mm to (170.7, 63.6)
Routing:
- net GND: vias 212 -> 36
- net /POWER_CTRL/SUPPLY: vias 193 -> 7
