File: gsvesc.sch (KiCad schematic (older format))
At the start: 25 parts

Commit message: SCM Fertig
Parts:
- C1: renamed from C?; footprint (none) -> Capacitor_SMD:C_0805_2012Metric
- C2: renamed from C?; value C -> 100n; footprint (none) -> Capacitor_SMD:C_0805_2012Metric
- D1, D2, D3: renamed from D?; footprint (none) -> LED_SMD:LED_0805_2012Metric
- J1, J2, J3: renamed from J?; footprint (none) -> Connector_JST:JST_PH_B6B-PH-K_1x06_P2.00mm_Vertical
- J4: renamed from J?; footprint (none) -> Connector_PinHeader_2.54mm:PinHeader_1x05_P2.54mm_Vertical
- J5, J9: renamed from J?; footprint (none) -> Connector_JST:JST_PH_B3B-PH-K_1x03_P2.00mm_Vertical
- J7, J8: renamed from J?; footprint (none) -> Connector_Wire:SolderWirePad_1x01_Drill2.5mm
- R1, R10, R11, R2, R3, R4, R5, R6, R7, R8, R9: renamed from R?; footprint (none) -> Resistor_SMD:R_0805_2012Metric
- gave numbers to parts that had none: 1

Commit message: design finished gerber created
Parts:
- J7, J8: footprint Connector_Wire:SolderWirePad_1x01_Drill2.5mm -> Connector_Wire:SolderWirePad_1x01_SMD_5x10mm
Connections:
- no-connect marks 0 -> 7
Changed lines of the file:
@@
 F0 "DRV8301" 50
 F1 "gsvesc_drv.sch" 50
-F2 "INH_a" I L 5450 1550 50
+F2 "INH_A" I L 5450 1550 50
 F3 "INH_B" I L 5450 1650 50
 F4 "INH_C" I L 5450 1750 50
@@
 F15 "SENS_B" O L 5450 3100 50
 F16 "SENS_C" O L 5450 3200 50
-F17 "SENS_VBAT" O L 5450 3300 50
+F17 "SENSE_VBAT" O L 5450 3300 50
 F18 "VBAT" I R 6500 1550 50
 F19 "GH_A" O R 6500 2050 50
@@
 	6500 1550 7550 1550
 Wire Wire Line
-	8150 1550 8950 1550
+	8450 1550 8700 1550
 Wire Wire Line
 	4600 5100 5200 5100
@@
 F 0 "J7" H 10480 1592 50  0000 L CNN
 F 1 "BAT+" H 10480 1501 50  0000 L CNN
-F 2 "Connector_Wire:SolderWirePad_1x01_Drill2.5mm" H 10400 1550 50  0001 C CNN
+F 2 "Connector_Wire:SolderWirePad_1x01_SMD_5x10mm" H 10400 1550 50  0001 C CNN
 F 3 "~" H 10400 1550 50  0001 C CNN
 	1    10400 1550
@@
 F 0 "J8" H 10480 1892 50  0000 L CNN
 F 1 "BAT-" H 10480 1801 50  0000 L CNN
-F 2 "Connector_Wire:SolderWirePad_1x01_Drill2.5mm" H 10400 1850 50  0001 C CNN
+F 2 "Connector_Wire:SolderWirePad_1x01_SMD_5x10mm" H 10400 1850 50  0001 C CNN
 F 3 "~" H 10400 1850 50  0001 C CNN
 	1    10400 1850
@@
 	1    0    0    -1
 $EndComp
+NoConn ~ 1900 1900
+NoConn ~ 4600 4300
+NoConn ~ 4600 4400
+NoConn ~ 4600 4500
+NoConn ~ 4600 4600
+NoConn ~ 4600 4700
+NoConn ~ 1700 5300
+$Comp
+L power:PWR_FLAG #FLG0102
+U 1 1 5C34D8D2
+P 8700 1550
+F 0 "#FLG0102" H 8700 1625 50  0001 C CNN
+F 1 "PWR_FLAG" V 8700 1678 50  0000 L CNN
+F 2 "" H 8700 1550 50  0001 C CNN
+F 3 "~" H 8700 1550 50  0001 C CNN
+	1    8700 1550
+	1    0    0    -1
+$EndComp
+Connection ~ 8700 1550
+Wire Wire Line
+	8700 1550 8950 1550
 $EndSCHEMATC

Commit message: Revision 2.0a
Connections:
- net MCU/USB_D+: now also R3.1; no longer R2.1
- net MCU/USB_D-: now also R2.1; no longer R3.1
Changed lines of the file:
@@
 	0    1    1    0
 $EndComp
-Wire Wire Line
-	2350 1700 3250 1700
 $Comp
 L Device:R R3
@@
 	0    1    1    0
 $EndComp
-Wire Wire Line
-	2350 1800 3250 1800
 Wire Wire Line
 	1900 1500 2050 1500
@@
 Wire Wire Line
 	8700 1550 8950 1550
+Wire Wire Line
+	2350 1700 2800 1700
+Wire Wire Line
+	2800 1700 2800 1800
+Wire Wire Line
+	2800 1800 3250 1800
+Wire Wire Line
+	2700 1800 2700 1900
+Wire Wire Line
+	2700 1900 2950 1900
+Wire Wire Line
+	2950 1900 2950 1700
+Wire Wire Line
+	2950 1700 3250 1700
+Wire Wire Line
+	2350 1800 2700 1800
 $EndSCHEMATC

Commit message: fix some bugs
Connections:
- net MCU/USB_D+: now also R2.1; no longer R3.1
- net MCU/USB_D-: now also R3.1; no longer R2.1
Changed lines of the file:
@@
 	8700 1550 8950 1550
 Wire Wire Line
-	2350 1700 2800 1700
+	2350 1800 3250 1800
 Wire Wire Line
-	2800 1700 2800 1800
-Wire Wire Line
-	2800 1800 3250 1800
-Wire Wire Line
-	2700 1800 2700 1900
-Wire Wire Line
-	2700 1900 2950 1900
-Wire Wire Line
-	2950 1900 2950 1700
-Wire Wire Line
-	2950 1700 3250 1700
-Wire Wire Line
-	2350 1800 2700 1800
+	2350 1700 3250 1700
 $EndSCHEMATC

Commit message: test
Parts:
- removed J9: Conn_01x03, Connector_JST:JST_PH_B3B-PH-K_1x03_P2.00mm_Vertical, symbol Connector_Generic:Conn_01x03
Connections:
- no-connect marks 7 -> 11
Changed lines of the file:
@@
 Title "GSVESC - DC Motor Controler"
 Date "2018-11-11"
-Rev "2.0"
+Rev "3.0"
 Comp ""
 Comment1 ""
@@
 F36 "CURRENT_3" I R 4600 4000 50
 F37 "ADC_TEMP" I R 4600 4100 50
-F38 "NRF_MISO" I R 4600 5100 50
-F39 "NRF_MOSI" O R 4600 5200 50
-F40 "NRF_SCK" O R 4600 5300 50
-F41 "NRF_CSN" O R 4600 5400 50
-F42 "HALL_1" I L 3250 3050 50
-F43 "HALL_2" I L 3250 3150 50
-F44 "HALL_3" I L 3250 3250 50
-F45 "PB8" I R 4600 4500 50
-F46 "PB9" I R 4600 4600 50
-F47 "PC5" I R 4600 4700 50
-F48 "PA15" I R 4600 4300 50
-F49 "PB2" I R 4600 4400 50
+F38 "HALL_1" I L 3250 3050 50
+F39 "HALL_2" I L 3250 3150 50
+F40 "HALL_3" I L 3250 3250 50
+F41 "PB8" I R 4600 4700 50
+F42 "PB9" I R 4600 4800 50
+F43 "PC5" I R 4600 5000 50
+F44 "PA15" I R 4600 4300 50
+F45 "PB2" I R 4600 4400 50
+F46 "PB3" I R 4600 4500 50
+F47 "PB4" I R 4600 4600 50
+F48 "P_UART_TX" I R 4600 5300 50
+F49 "P_UART_RX" I R 4600 5400 50
+F50 "PB12" I R 4600 4900 50
+F51 "PD2" I R 4600 5100 50
 $EndSheet
 $Comp
@@
 F1 "gsvesc_pwrctrl.sch" 50
 F2 "VBAT" O L 8950 1550 50
-F3 "ESC_IN" I R 9850 2500 50
-F4 "5V_CTRL" O R 9850 2400 50
-F5 "SUPPLY" I R 9850 1550 50
+F3 "SUPPLY" I R 9850 1550 50
 $EndSheet
 $Sheet
@@
 F0 "NRF" 50
 F1 "gsvesc_nrf.sch" 50
-F2 "MISO" O L 5200 5100 50
-F3 "MOSI" I L 5200 5200 50
-F4 "SCLK" I L 5200 5300 50
-F5 "CS" I L 5200 5400 50
+F2 "NRF_TX" I L 5200 5300 50
+F3 "NRF_RX" I L 5200 5400 50
 $EndSheet
 $Comp
@@
 Wire Wire Line
 	8450 1550 8700 1550
-Wire Wire Line
-	4600 5100 5200 5100
-Wire Wire Line
-	5200 5200 4600 5200
-Wire Wire Line
-	4600 5300 5200 5300
-Wire Wire Line
-	5200 5400 4600 5400
-$Comp
-L Connector_Generic:Conn_01x03 J9
-U 1 1 5BEDC794
-P 10400 3150
-F 0 "J9" H 10320 2825 50  0000 C CNN
-F 1 "Conn_01x03" H 10320 2916 50  0000 C CNN
-F 2 "Connector_JST:JST_PH_B3B-PH-K_1x03_P2.00mm_Vertical" H 10400 3150 50  0001 C CNN
-F 3 "~" H 10400 3150 50  0001 C CNN
-	1    10400 3150
-	1    0    0    -1
-$EndComp
-Wire Wire Line
-	9850 2500 9950 2500
-Wire Wire Line
-	9950 2500 9950 3150
-Wire Wire Line
-	9950 3150 10200 3150
-$Comp
-L power:GND #PWR018
-U 1 1 5BEEC336
-P 9850 3250
-F 0 "#PWR018" H 9850 3000 50  0001 C CNN
-F 1 "GND" V 9855 3122 50  0000 R CNN
-F 2 "" H 9850 3250 50  0001 C CNN
-F 3 "" H 9850 3250 50  0001 C CNN
-	1    9850 3250
-	0    1    1    0
-$EndComp
-Wire Wire Line
-	9850 3250 10200 3250
-Wire Wire Line
-	9850 2400 10050 2400
-Wire Wire Line
-	10050 2400 10050 3050
-Wire Wire Line
-	10050 3050 10200 3050
 $Comp
 L Connector_Generic:Conn_01x01 J7
@@
 Wire Wire Line
 	2350 1700 3250 1700
+NoConn ~ 4600 4800
+NoConn ~ 4600 4900
+NoConn ~ 4600 5000
+NoConn ~ 4600 5100
+Wire Wire Line
+	4600 5300 5200 5300
+Wire Wire Line
+	4600 5400 5200 5400
 $EndSCHEMATC

Commit message: gsesc v3, work in progress
Parts:
- added C45, C46: 680u/80V, Capacitor_THT:CP_Radial_D12.5mm_P5.00mm, symbol Device:CP
- added H1, H2, H3: MountingHole, MountingHole:MountingHole_3.2mm_M3, symbol Mechanical:MountingHole
- J7, J8: footprint Connector_Wire:SolderWirePad_1x01_SMD_5x10mm -> gsvesc:TestPoint_Pad_5.0x5.0mm
Connections:
- net POWER_CTRL/SUPPLY is gone; now on net POWER/VBAT: J7.1 (Pin_1)
- net GND: now also C45.2, C46.2
- net MCU/PC5: now also J3.3 (Pin_3)
- net POWER/VBAT: now also C45.1, C46.1
- no-connect marks 11 -> 3
Other:
- note added: "based on Benjamin Vedders VESC 6"
Changed lines of the file:
@@
 $Descr A4 11693 8268
 encoding utf-8
-Sheet 1 6
-Title "GSVESC - DC Motor Controler"
+Sheet 1 5
+Title "GSESC - DC Motor Controler"
 Date "2018-11-11"
 Rev "3.0"
@@
 F39 "HALL_2" I L 3250 3150 50
 F40 "HALL_3" I L 3250 3250 50
-F41 "PB8" I R 4600 4700 50
-F42 "PB9" I R 4600 4800 50
-F43 "PC5" I R 4600 5000 50
-F44 "PA15" I R 4600 4300 50
-F45 "PB2" I R 4600 4400 50
-F46 "PB3" I R 4600 4500 50
-F47 "PB4" I R 4600 4600 50
-F48 "P_UART_TX" I R 4600 5300 50
-F49 "P_UART_RX" I R 4600 5400 50
-F50 "PB12" I R 4600 4900 50
-F51 "PD2" I R 4600 5100 50
+F41 "PC5" I L 3250 5300 50
+F42 "PA15" I R 4600 4300 50
+F43 "PB2" I R 4600 5000 50
+F44 "PB3" I R 4600 5100 50
+F45 "PB4" I R 4600 5200 50
+F46 "P_UART_TX" I R 4600 5300 50
+F47 "P_UART_RX" I R 4600 5400 50
+F48 "PB12" I R 4600 4400 50
+F49 "CURR_FILTER_ON" O R 4600 3700 50
 $EndSheet
 $Comp
@@
 F18 "TEMP" O L 7550 4100 50
 F19 "VBAT" I R 8450 1550 50
-$EndSheet
-$Sheet
-S 8950 1450 900  1200
-U 5BECFBCA
-F0 "POWER_CTRL" 50
-F1 "gsvesc_pwrctrl.sch" 50
-F2 "VBAT" O L 8950 1550 50
-F3 "SUPPLY" I R 9850 1550 50
+F20 "CURR_FILTER" I L 7550 3700 50
 $EndSheet
 $Sheet
@@
 F2 "NRF_TX" I L 5200 5300 50
 F3 "NRF_RX" I L 5200 5400 50
+F4 "GPIO1" I L 5200 5000 50
+F5 "GPIO2" I L 5200 5100 50
+F6 "GPIO3" I L 5200 5200 50
 $EndSheet
 $Comp
@@
 Wire Wire Line
 	6500 1550 7550 1550
-Wire Wire Line
-	8450 1550 8700 1550
 $Comp
 L Connector_Generic:Conn_01x01 J7
@@
 F 0 "J7" H 10480 1592 50  0000 L CNN
 F 1 "BAT+" H 10480 1501 50  0000 L CNN
-F 2 "Connector_Wire:SolderWirePad_1x01_SMD_5x10mm" H 10400 1550 50  0001 C CNN
+F 2 "gsvesc:TestPoint_Pad_5.0x5.0mm" H 10400 1550 50  0001 C CNN
 F 3 "~" H 10400 1550 50  0001 C CNN
 	1    10400 1550
@@
 F 0 "J8" H 10480 1892 50  0000 L CNN
 F 1 "BAT-" H 10480 1801 50  0000 L CNN
-F 2 "Connector_Wire:SolderWirePad_1x01_SMD_5x10mm" H 10400 1850 50  0001 C CNN
+F 2 "gsvesc:TestPoint_Pad_5.0x5.0mm" H 10400 1850 50  0001 C CNN
 F 3 "~" H 10400 1850 50  0001 C CNN
 	1    10400 1850
 	1    0    0    -1
 $EndComp
-Wire Wire Line
-	9850 1550 10200 1550
 Wire Wire Line
 	10200 1850 10200 1950
@@
 NoConn ~ 4600 4300
 NoConn ~ 4600 4400
-NoConn ~ 4600 4500
-NoConn ~ 4600 4600
-NoConn ~ 4600 4700
-NoConn ~ 1700 5300
 $Comp
 L power:PWR_FLAG #FLG0102
@@
 Connection ~ 8700 1550
 Wire Wire Line
-	8700 1550 8950 1550
-Wire Wire Line
 	2350 1800 3250 1800
 Wire Wire Line
 	2350 1700 3250 1700
-NoConn ~ 4600 4800
-NoConn ~ 4600 4900
-NoConn ~ 4600 5000
-NoConn ~ 4600 5100
 Wire Wire Line
 	4600 5300 5200 5300
 Wire Wire Line
 	4600 5400 5200 5400
+Wire Wire Line
+	4600 3700 7550 3700
+$Comp
+L power:GND #PWR?
+U 1 1 5DF681DF
+P 8900 2400
+AR Path="/5BECFBCA/5DF681DF" Ref="#PWR?"  Part="1"
+AR Path="/5DF681DF" Ref="#PWR0110"  Part="1"
+F 0 "#PWR0110" H 8900 2150 50  0001 C CNN
+F 1 "GND" H 8905 2227 50  0000 C CNN
+F 2 "" H 8900 2400 50  0001 C CNN
+F 3 "" H 8900 2400 50  0001 C CNN
+	1    8900 2400
+	1    0    0    -1
+$EndComp
+Wire Wire Line
+	8900 2250 8900 2400
+Wire Wire Line
+	8900 2250 9650 2250
+Wire Wire Line
+	9650 2250 9650 2000
+Wire Wire Line
+	8900 2000 8900 2250
+Wire Wire Line
+	8900 1700 8900 1550
+Wire Wire Line
+	9650 1550 9650 1700
+$Comp
+L Device:CP C?
+U 1 1 5DF681EB
+P 9650 1850
+AR Path="/5BECFBCA/5DF681EB" Ref="C?"  Part="1"
+AR Path="/5DF681EB" Ref="C46"  Part="1"
+F 0 "C46" H 9768 1896 50  0000 L CNN
+F 1 "680u/80V" H 9768 1805 50  0000 L CNN
+F 2 "Capacitor_THT:CP_Radial_D12.5mm_P5.00mm" H 9688 1700 50  0001 C CNN
+F 3 "~" H 9650 1850 50  0001 C CNN
+	1    9650 1850
+	1    0    0    -1
+$EndComp
+$Comp
+L Device:CP C?
+U 1 1 5DF681F2
+P 8900 1850
+AR Path="/5BECFBCA/5DF681F2" Ref="C?"  Part="1"
+AR Path="/5DF681F2" Ref="C45"  Part="1"
+F 0 "C45" H 9018 1896 50  0000 L CNN
+F 1 "680u/80V" H 9018 1805 50  0000 L CNN
+F 2 "Capacitor_THT:CP_Radial_D12.5mm_P5.00mm" H 8938 1700 50  0001 C CNN
+F 3 "~" H 8900 1850 50  0001 C CNN
+	1    8900 1850
+	1    0    0    -1
+$EndComp
+Connection ~ 9650 1550
+Wire Wire Line
+	9650 1550 10200 1550
+Connection ~ 8900 2250
+Connection ~ 8900 1550
+Wire Wire Line
+	8900 1550 9650 1550
+Wire Wire Line
+	8700 1550 8900 1550
+Wire Wire Line
+	8450 1550 8700 1550
+Wire Wire Line
+	4600 5000 5200 5000
+Wire Wire Line
+	4600 5100 5200 5100
+Wire Wire Line
+	4600 5200 5200 5200
+$Comp
+L Mechanical:MountingHole H1
+U 1 1 5E309F9C
+P 10500 5650
+F 0 "H1" H 10600 5696 50  0000 L CNN
+F 1 "MountingHole" H 10600 5605 50  0000 L CNN
+F 2 "MountingHole:MountingHole_3.2mm_M3" H 10500 5650 50  0001 C CNN
+F 3 "~" H 10500 5650 50  0001 C CNN
+	1    10500 5650
+	1    0    0    -1
+$EndComp
+$Comp
+L Mechanical:MountingHole H2
+U 1 1 5E30A04A
+P 10500 5900
+F 0 "H2" H 10600 5946 50  0000 L CNN
+F 1 "MountingHole" H 10600 5855 50  0000 L CNN
+F 2 "MountingHole:MountingHole_3.2mm_M3" H 10500 5900 50  0001 C CNN
+F 3 "~" H 10500 5900 50  0001 C CNN
+	1    10500 5900
+	1    0    0    -1
+$EndComp
+$Comp
+L Mechanical:MountingHole H3
+U 1 1 5E30A09C
+P 10500 6150
+F 0 "H3" H 10600 6196 50  0000 L CNN
+F 1 "MountingHole" H 10600 6105 50  0000 L CNN
+F 2 "MountingHole:MountingHole_3.2mm_M3" H 10500 6150 50  0001 C CNN
+F 3 "~" H 10500 6150 50  0001 C CNN
+	1    10500 6150
+	1    0    0    -1
+$EndComp
+Wire Wire Line
+	1700 5300 3250 5300
+Text Notes 7200 7050 0    79   ~ 0
+based on Benjamin Vedders VESC 6
 $EndSCHEMATC

Commit message: library wieder im projektordner
Parts:
- H1, H2, H3: footprint MountingHole:MountingHole_3.2mm_M3 -> MountingHole:MountingHole_4.3mm_M4
Changed lines of the file:
@@
 F 0 "H1" H 10600 5696 50  0000 L CNN
 F 1 "MountingHole" H 10600 5605 50  0000 L CNN
-F 2 "MountingHole:MountingHole_3.2mm_M3" H 10500 5650 50  0001 C CNN
+F 2 "MountingHole:MountingHole_4.3mm_M4" H 10500 5650 50  0001 C CNN
 F 3 "~" H 10500 5650 50  0001 C CNN
 	1    10500 5650
@@
 F 0 "H2" H 10600 5946 50  0000 L CNN
 F 1 "MountingHole" H 10600 5855 50  0000 L CNN
-F 2 "MountingHole:MountingHole_3.2mm_M3" H 10500 5900 50  0001 C CNN
+F 2 "MountingHole:MountingHole_4.3mm_M4" H 10500 5900 50  0001 C CNN
 F 3 "~" H 10500 5900 50  0001 C CNN
 	1    10500 5900
@@
 F 0 "H3" H 10600 6196 50  0000 L CNN
 F 1 "MountingHole" H 10600 6105 50  0000 L CNN
-F 2 "MountingHole:MountingHole_3.2mm_M3" H 10500 6150 50  0001 C CNN
+F 2 "MountingHole:MountingHole_4.3mm_M4" H 10500 6150 50  0001 C CNN
 F 3 "~" H 10500 6150 50  0001 C CNN
 	1    10500 6150

Commit message: Update
Parts:
- C45, C46: value 680u/80V -> 680u/63V
- H1, H2, H3: footprint MountingHole:MountingHole_4.3mm_M4 -> MountingHole:MountingHole_3.2mm_M3
Changed lines of the file:
@@
 AR Path="/5DF681EB" Ref="C46"  Part="1"
 F 0 "C46" H 9768 1896 50  0000 L CNN
-F 1 "680u/80V" H 9768 1805 50  0000 L CNN
+F 1 "680u/63V" H 9768 1805 50  0000 L CNN
 F 2 "Capacitor_THT:CP_Radial_D12.5mm_P5.00mm" H 9688 1700 50  0001 C CNN
 F 3 "~" H 9650 1850 50  0001 C CNN
@@
 AR Path="/5DF681F2" Ref="C45"  Part="1"
 F 0 "C45" H 9018 1896 50  0000 L CNN
-F 1 "680u/80V" H 9018 1805 50  0000 L CNN
+F 1 "680u/63V" H 9018 1805 50  0000 L CNN
 F 2 "Capacitor_THT:CP_Radial_D12.5mm_P5.00mm" H 8938 1700 50  0001 C CNN
 F 3 "~" H 8900 1850 50  0001 C CNN
@@
 F 0 "H1" H 10600 5696 50  0000 L CNN
 F 1 "MountingHole" H 10600 5605 50  0000 L CNN
-F 2 "MountingHole:MountingHole_4.3mm_M4" H 10500 5650 50  0001 C CNN
+F 2 "MountingHole:MountingHole_3.2mm_M3" H 10500 5650 50  0001 C CNN
 F 3 "~" H 10500 5650 50  0001 C CNN
 	1    10500 5650
@@
 F 0 "H2" H 10600 5946 50  0000 L CNN
 F 1 "MountingHole" H 10600 5855 50  0000 L CNN
-F 2 "MountingHole:MountingHole_4.3mm_M4" H 10500 5900 50  0001 C CNN
+F 2 "MountingHole:MountingHole_3.2mm_M3" H 10500 5900 50  0001 C CNN
 F 3 "~" H 10500 5900 50  0001 C CNN
 	1    10500 5900
@@
 F 0 "H3" H 10600 6196 50  0000 L CNN
 F 1 "MountingHole" H 10600 6105 50  0000 L CNN
-F 2 "MountingHole:MountingHole_4.3mm_M4" H 10500 6150 50  0001 C CNN
+F 2 "MountingHole:MountingHole_3.2mm_M3" H 10500 6150 50  0001 C CNN
 F 3 "~" H 10500 6150 50  0001 C CNN
 	1    10500 6150
