File: gsvesc.kicad_pcb (KiCad board)
At the start: 4 copper layers, 111 x 111 mm, 126 parts, among them J1 Conn_01x06, J10 PHASE_C, J11 PHASE_B, J12 NTC, J14 Conn_02x04_Odd_Even, J2 Conn_01x06, J3 Conn_01x06, J4 Conn_01x05, J5 Conn_01x03, J6 USB_B_Mini, J7 BAT+, J8 BAT-, J9 PHASE_A, Q1 TPH2R506PL, Q2 TPH2R506PL, Q3 TPH2R506PL, Q4 TPH2R506PL, Q5 TPH2R506PL, Q6 TPH2R506PL, U1 STM32F405RGTx, U2 IRU1010-33, U3 DCA56_6P35X3P61, U4 INA240A3, U5 INA240A3, U6 INA240A3, U7 TSOP-5, U8 TSOP-5, U9 TSOP-5, Y1 ABM3B 8MHz

Commit message: V4 pre
Parts:
- added D6: B5819W, Diode_SMD:D_SOD-123, F.Cu at (114.2, 149.5)
- added D7: B5819W, Diode_SMD:D_SOD-123, F.Cu at (103.1, 141.9)
- added J13: Conn_01x02, gsvesc:2pad_smd_testpin, F.Cu at (80.7, 119.8)
- added L2: 15u0, Inductor_SMD:L_7.3x7.3_H4.5, F.Cu at (91.5, 132.0)
- added R27: 10k0, Resistor_SMD:R_0805_2012Metric, F.Cu at (87.8, 138.1)
- added R34: 5k90, Resistor_SMD:R_0805_2012Metric, F.Cu at (90.4, 142.2)
- added U10: LM5008MM, Package_SO:MSOP-8_3x3mm_P0.65mm, F.Cu at (112.8, 143.4)
- added U11: M74VHC1GT66DTT1G, gsvesc:M74VHC1GT66DTT1G, F.Cu at (63.1, 97.3)
- added U12: LM5107, Package_SO:SOIC-8_3.9x4.9mm_P1.27mm, F.Cu at (62.2, 91.0)
- added U13: M74VHC1GT66DTT1G, gsvesc:M74VHC1GT66DTT1G, F.Cu at (72.2, 97.4)
- added U14: TPS5430DDA, Package_SO:TI_SO-PowerPAD-8_ThermalVias, F.Cu at (95.5, 139.5)
- added U15: LM5107, Package_SO:SOIC-8_3.9x4.9mm_P1.27mm, F.Cu at (71.6, 91.0)
- C1: value 100N -> 100n
- C10, C11, C12, C13, C15, C42, C6, C7, C8, C9: value 10u0/16V -> 10u0/25V
- C14, C24, C41: value 1n00 -> 10n0
- C16: value 100n -> 10u0/75V; footprint Capacitor_SMD:C_0805_2012Metric -> Capacitor_SMD:C_1210_3225Metric
- C17: value 6n80 -> 100n
- C18, C19, C21: value 10u0/16V -> 100n
- C20: value 150p -> 10n0
- C22: value 22n0 -> 10u0/25V
- C23: value 10u0/16V -> 10n0
- C26: value 10u0/75V -> 22u0/25V; footprint Capacitor_SMD:C_1210_3225Metric -> Capacitor_SMD:C_0805_2012Metric
- C28: value 15n0 -> 10u0/25V
- C29: value 220n -> 10u0/25V
- C30: value 220n -> 100n
- C31: value 220n -> 10n0
- C32: value 10u0/75V -> 100n; footprint Capacitor_SMD:C_1210_3225Metric -> Capacitor_SMD:C_0805_2012Metric
- C33: value 10u0/16V -> 100u; footprint Capacitor_SMD:C_0805_2012Metric -> Capacitor_Tantalum_SMD:CP_EIA-3528-21_Kemet-B
- C34: value 100u/16V -> 100u; footprint Capacitor_Tantalum_SMD:CP_EIA-3216-18_Kemet-A -> Capacitor_Tantalum_SMD:CP_EIA-3528-21_Kemet-B
- D4: value B360_SMA -> SS210
- D5: value SMBJ6.0CA -> SS210; footprint Diode_SMD:D_SMB -> Diode_SMD:D_SMA
- J1, J2, J3: footprint Connector_JST:JST_PH_B6B-PH-SM4-TB_1x06-1MP_P2.00mm_Vertical -> Connector_JST:JST_SH_BM06B-SRSS-TB_1x06-1MP_P1.00mm_Vertical
- J12: footprint Connector_PinHeader_2.54mm:PinHeader_2x01_P2.54mm_Vertical -> gsvesc:2pad_smd_testpin
- J5: footprint Connector_JST:JST_PH_B3B-PH-SM4-TB_1x03-1MP_P2.00mm_Vertical -> Connector_JST:JST_SH_BM03B-SRSS-TB_1x03-1MP_P1.00mm_Vertical
- L1: value 22u -> 470u; footprint Inductor_SMD:L_Bourns_SRN6045TA -> Inductor_SMD:L_12x12mm_H6mm
- R12: value 3k31 -> 680k
- R13: value 18k2 -> 56k0
- R14: value 15k0 -> 2k70
- R15: value 10k0 -> 680k
- R16: value 221k -> 10k0
- R17, R19, R21: value 39k0 -> 56k0
- R18, R20, R22: value 2k21 -> 2k70
- R23: value 39k0 -> 2k70
- R24: value 2k21 -> 4R75
- R38: value 100k -> 4R75
- R39: value 3k2 -> 4R75
- R4, R6, R7: value 2K21 -> 2k70
- U2: value IRU1010-33 -> M74VHC1GT66DTT1G; footprint Package_TO_SOT_SMD:SOT-223 -> gsvesc:M74VHC1GT66DTT1G
- U3: value DCA56_6P35X3P61 -> LM5107; footprint gsvesc:DRV8301DCAR -> Package_SO:SOIC-8_3.9x4.9mm_P1.27mm
- U7, U8, U9: value TSOP-5 -> M74VHC1GT66DTT1G
- moved C16 81.1 mm to (117.4, 147.1), turned to 270 degrees
- moved D4 78.7 mm to (121.8, 135.7), turned to 90 degrees
- moved C17 70.0 mm to (118.2, 141.9)
- moved R12 68.8 mm to (120.4, 146.5)
- moved R23 68.8 mm to (108.9, 147.7), turned to 180 degrees
- moved C20 66.0 mm to (115.8, 141.8)
- moved L1 65.9 mm to (112.0, 132.8), turned to 0 degrees
- moved C23 65.2 mm to (108.9, 145.5)
- moved D5 63.3 mm to (97.5, 132.7)
- moved C28 59.1 mm to (102.9, 139.0), turned to 0 degrees
- moved R16 59.0 mm to (108.9, 143.3), turned to 0 degrees
- moved R38 53.4 mm to (102.9, 131.8), turned to 0 degrees
- moved R39 52.7 mm to (102.8, 134.2), turned to 0 degrees
- moved R15 52.3 mm to (108.8, 141.2), turned to 180 degrees
- moved C19 52.1 mm to (111.8, 148.8)
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Connections:
- C15 pad 1: Net-(C15-Pad1) -> +12V
- C16 pad 1: +5V -> VBAT
- C17 pad 1: GND -> VBAT
- C17 pad 2: Net-(C17-Pad2) -> GND
- C18 pad 1: Net-(C15-Pad1) -> Net-(C18-Pad1)
- C18 pad 2: GND -> /Driver/SENS_A
- C20 pad 1: GND -> Net-(C20-Pad1)
- C21 pad 2: GND -> /Driver/SH_A
- C22 pad 1: Net-(C22-Pad1) -> +12V
- C22 pad 2: Net-(C22-Pad2) -> GND
- C23 pad 1: VCC -> Net-(C23-Pad1)
- C23 pad 2: GND -> Net-(C23-Pad2)
- C25 pad 1: VCC -> Net-(C25-Pad1)
- C25 pad 2: GND -> /Driver/SENS_B
- C26 pad 1: /DRV8301/VBAT -> +12V
- C27 pad 2: Net-(C27-Pad2) -> /Driver/SH_B
- C28 pad 1: GND -> +12V
- C28 pad 2: Net-(C28-Pad2) -> GND
- C29 pad 1: /DRV8301/SH_A -> +12V
- C29 pad 2: Net-(C29-Pad2) -> GND
- C30 pad 1: /DRV8301/SH_B -> Net-(C30-Pad1)
- C30 pad 2: Net-(C30-Pad2) -> /Driver/SENS_C
- C31 pad 1: /DRV8301/SH_C -> Net-(C31-Pad1)
- C32 pad 1: /DRV8301/VBAT -> Net-(C32-Pad1)
- C32 pad 2: GND -> /Driver/SH_C
- C33 pad 1: +5V -> VCC
- C34 pad 1: +5V -> VCC
- C36 pad 1: /DRV8301/VBAT -> VBAT
- C37 pad 1: /DRV8301/VBAT -> VBAT
- C38 pad 1: /DRV8301/VBAT -> VBAT
- C39 pad 1: /DRV8301/VBAT -> VBAT
- C43 pad 1: /DRV8301/VBAT -> VBAT
- C44 pad 1: /DRV8301/VBAT -> VBAT
- D4 pad 1: Net-(C27-Pad1) -> Net-(C20-Pad2)
- D5 pad 1: +5V -> Net-(C31-Pad1)
- J7 pad 1: /DRV8301/VBAT -> VBAT
- L1 pad 1: Net-(C27-Pad1) -> Net-(C23-Pad1)
- L1 pad 2: +5V -> Net-(C20-Pad2)
- Q1 pad 1: /DRV8301/VBAT -> VBAT
- Q1 pad 3: /DRV8301/SH_A -> /Driver/SH_A
- Q2 pad 1: /DRV8301/SH_A -> /Driver/SH_A
- Q3 pad 1: /DRV8301/VBAT -> VBAT
- Q3 pad 3: /DRV8301/SH_C -> /Driver/SH_C
- Q4 pad 1: /DRV8301/SH_C -> /Driver/SH_C
- Q5 pad 1: /DRV8301/VBAT -> VBAT
- Q5 pad 3: /DRV8301/SH_B -> /Driver/SH_B
- Q6 pad 1: /DRV8301/SH_B -> /Driver/SH_B
- R12 pad 1: GND -> /Driver/EXT_OFF
- R12 pad 2: Net-(R12-Pad2) -> VBAT
- R13 pad 1: Net-(R12-Pad2) -> /Driver/SH_A
- R13 pad 2: +5V -> /Driver/SENS_A
- R14 pad 1: Net-(C17-Pad2) -> GND
- R14 pad 2: Net-(C20-Pad2) -> /Driver/SENS_A
- R15 pad 1: GND -> Net-(R15-Pad1)
- R15 pad 2: Net-(R15-Pad2) -> GND
- R16 pad 1: GND -> Net-(C23-Pad1)
- R16 pad 2: Net-(R16-Pad2) -> Net-(C23-Pad2)
- R17 pad 1: /DRV8301/VBAT -> /Driver/SH_B
- R17 pad 2: /MCU/AN_IN -> /Driver/SENS_B
- R18 pad 2: /MCU/AN_IN -> /Driver/SENS_B
- R19 pad 1: /DRV8301/SH_A -> /Driver/SH_C
- R19 pad 2: /DRV8301/SENS_A -> /Driver/SENS_C
- R20 pad 2: /DRV8301/SENS_A -> /Driver/SENS_C
- R21 pad 1: /DRV8301/SH_B -> VBAT
- R21 pad 2: /DRV8301/SENS_B -> /MCU/AN_IN
- R22 pad 2: /DRV8301/SENS_B -> /MCU/AN_IN
- R23 pad 1: /DRV8301/SH_C -> Net-(C23-Pad2)
- R23 pad 2: /DRV8301/SENS_C -> GND
- R24 pad 1: GND -> +12V
- R24 pad 2: /DRV8301/SENS_C -> Net-(C23-Pad1)
- R25 pad 2: /DRV8301/GH_C -> /Driver/GH_C
- R26 pad 2: /DRV8301/GL_C -> /Driver/GL_C
- R28 pad 2: /DRV8301/GH_A -> /Driver/GH_A
- R31 pad 2: /DRV8301/SH_C -> /Driver/SH_C
- R32 pad 2: /DRV8301/GL_A -> /Driver/GL_A
- R38 pad 1: /DRV8301/VBAT -> +12V
- R38 pad 2: Net-(R38-Pad2) -> Net-(C23-Pad1)
- R39 pad 1: Net-(R38-Pad2) -> +12V
- R39 pad 2: GND -> Net-(C23-Pad1)
- R42 pad 2: /DRV8301/GH_B -> /Driver/GH_B
- R43 pad 2: /DRV8301/GL_B -> /Driver/GL_B
- R45 pad 2: /DRV8301/SH_A -> /Driver/SH_A
- R46 pad 2: /DRV8301/SH_B -> /Driver/SH_B
- U1 pad 14: /DRV8301/SENS_A -> /Driver/SENS_A
- U1 pad 15: /DRV8301/SENS_B -> /Driver/SENS_B
- U1 pad 16: /DRV8301/SENS_C -> /Driver/SENS_C
- U1 pad 34: /DRV8301/INL_A -> /MCU/L1
- U1 pad 35: /DRV8301/INL_B -> /MCU/L2
- U1 pad 36: /DRV8301/INL_C -> /MCU/L3
- U1 pad 40: /DRV8301/CS -> /Driver/SENS_FILTER
- U1 pad 51: /DRV8301/SCLK -> Net-(U1-Pad51)
- U1 pad 52: /DRV8301/SDO -> Net-(U1-Pad52)
- U1 pad 53: /DRV8301/SDI -> Net-(U1-Pad53)
- U1 pad 57: /DRV8301/EN_GATE -> Net-(U1-Pad57)
- U1 pad 62: /DRV8301/FAULT -> Net-(U1-Pad62)
- U2 pad 1: GND -> Net-(C18-Pad1)
- U2 pad 2: VCC -> GND
- U2 pad 3: +5V -> GND
- U2 pad 4: VCC -> /Driver/SENS_FILTER
- U3 pad 1: Net-(R16-Pad2) -> +12V
- U3 pad 2: Net-(C20-Pad2) -> /MCU/H1
- U3 pad 3: Net-(R12-Pad2) -> /MCU/L1
- U3 pad 4: Net-(U3-Pad4) -> GND
- U3 pad 5: Net-(U3-Pad5) -> /Driver/GL_A
- U3 pad 6: /DRV8301/FAULT -> /Driver/SH_A
- U3 pad 7: Net-(R15-Pad2) -> /Driver/GH_A
- U3 pad 8: /DRV8301/CS -> Net-(C21-Pad1)
- U4 pad 3: /DRV8301/SH_A -> /Driver/SH_A
- U5 pad 3: /DRV8301/SH_C -> /Driver/SH_C
- U6 pad 3: /DRV8301/SH_B -> /Driver/SH_B
Routing:
- net /DRV8301/GH_C: track 66.0 -> 0.00 mm, vias 2 -> 0
- net /DRV8301/SH_C: track 61.7 -> 0.00 mm, vias 35 -> 0
- net /DRV8301/GL_C: track 56.0 -> 0.00 mm, vias 2 -> 0
- net /Driver/SH_C: track 0.00 -> 55.3 mm, vias 0 -> 40
- net /Driver/GH_C: track 0.00 -> 53.4 mm, vias 0 -> 2
- net /DRV8301/SH_B: track 49.7 -> 0.00 mm, vias 45 -> 0
- net /Driver/SH_B: track 0.00 -> 48.8 mm, vias 0 -> 49
- net /POWER/CURR_FILTER: track 157.5 -> 109.7 mm
- net /DRV8301/SENS_B: track 45.5 -> 0.00 mm, vias 2 -> 0
- net /DRV8301/GH_B: track 45.3 -> 0.00 mm, vias 2 -> 0
- net /DRV8301/SENS_A: track 44.1 -> 0.00 mm, vias 2 -> 0
- net /DRV8301/GL_B: track 43.5 -> 0.00 mm, vias 2 -> 0
- net /DRV8301/SENS_C: track 43.3 -> 0.00 mm, vias 2 -> 0
- net /MCU/L1: track 0.00 -> 42.9 mm, vias 0 -> 3
- net /Driver/GL_C: track 0.00 -> 41.0 mm, vias 0 -> 2
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- added copper zone on B.Cu, net +12V
- added copper zone on F.Cu, net +12V
- added copper zone on B.Cu, net /Driver/SH_A
- added copper zone on F.Cu, net /Driver/SH_A
- added copper zone on In1.Cu, net /Driver/SH_A
- added copper zone on In2.Cu, net /Driver/SH_A
- added copper zone on B.Cu, net /Driver/SH_B
- added copper zone on F.Cu, net /Driver/SH_B
- added copper zone on In1.Cu, net /Driver/SH_B
- added copper zone on In2.Cu, net /Driver/SH_B
- added copper zone on B.Cu, net /Driver/SH_C
- added copper zone on F.Cu, net /Driver/SH_C
- added copper zone on In1.Cu, net /Driver/SH_C
- added copper zone on In2.Cu, net /Driver/SH_C
- added copper zone on F.Cu, net Net-(C20-Pad2)
- added copper zone on F.Cu, net Net-(C23-Pad1)
- added copper zone on F.Cu, net Net-(C31-Pad1)
- added copper zone on B.Cu, net VBAT
- added copper zone on F.Cu, net VBAT
- added copper zone on In1.Cu, net VBAT
- added copper zone on In2.Cu, net VBAT
- removed copper zone on B.Cu, net +5V
- removed copper zone on F.Cu, net +5V
- removed copper zone on B.Cu, net /DRV8301/SH_A
- removed copper zone on F.Cu, net /DRV8301/SH_A
- removed copper zone on In1.Cu, net /DRV8301/SH_A
- removed copper zone on In2.Cu, net /DRV8301/SH_A
- removed copper zone on B.Cu, net /DRV8301/SH_B
- removed copper zone on F.Cu, net /DRV8301/SH_B
- removed copper zone on In1.Cu, net /DRV8301/SH_B
- removed copper zone on In2.Cu, net /DRV8301/SH_B
- removed copper zone on B.Cu, net /DRV8301/SH_C
- removed copper zone on F.Cu, net /DRV8301/SH_C
- removed copper zone on In1.Cu, net /DRV8301/SH_C
- removed copper zone on In2.Cu, net /DRV8301/SH_C
- removed copper zone on B.Cu, net /DRV8301/VBAT
- removed copper zone on F.Cu, net /DRV8301/VBAT
- removed copper zone on In1.Cu, net /DRV8301/VBAT
- removed copper zone on In2.Cu, net /DRV8301/VBAT
- removed copper zone on F.Cu, net Net-(C27-Pad1)
Other:
- board text added: "2020 schardt@team-ctech.de"
- board text added: "GSVESC 4.0"
- board text added: "T-Motor"
- board text added: "T-PCB"
- board text removed: "GSVESC 3.0 2020 schardt@team-ctech.de"
