File: driver.sch (KiCad schematic (older format))
At the start: 53 parts, among them U10 LM5008MM, U11 SN74LVC1G66DBVR, U12 LM5107, U13 SN74LVC1G66DBVR, U14 TPS5430DDA, U15 LM5107, U2 SN74LVC1G66DBVR, U3 LM5107

Commit message: some bug fixes for next pcb-run
- Add JST connector for Motor Temp
- Remove USB 5V
- add correct footprint for D8,9,10
- add JST connector for external off
Parts:
- removed D7: B5819W, Diode_SMD:D_SOD-123, symbol Device:D_Schottky
- D10, D8, D9: symbol Device:D -> gsvesc:SMMBD914LT3G
Connections:
- net +12V: now also D10.1 (A), D8.1 (A), D9.1 (A); no longer D10.2 (A), D8.2 (A), D9.2 (A)
- net at C21.1, U3.8 (HB): now also D9.3 (K); no longer D9.1 (K)
- net at C27.1, U12.8 (HB): now also D10.3 (K); no longer D10.1 (K)
- net at C32.1, U15.8 (HB): now also D8.3 (K); no longer D8.1 (K)
Other:
- note removed: "USB powered"
Changed lines of the file:
@@
 	0    1    1    0
 $EndComp
-$Comp
-L Device:D_Schottky D7
-U 1 1 5E97305F
-P 7050 4900
-F 0 "D7" V 7100 4800 50  0000 C CNN
-F 1 "B5819W" V 7200 4700 50  0000 C CNN
-F 2 "Diode_SMD:D_SOD-123" H 7050 4900 50  0001 C CNN
-F 3 "~" H 7050 4900 50  0001 C CNN
-F 4 "C8598" H 7050 4900 50  0001 C CNN "LCSC"
-	1    7050 4900
-	0    -1   -1   0
-$EndComp
-Wire Wire Line
-	7050 4750 7050 4650
-Wire Wire Line
-	7050 4650 6400 4650
-$Comp
-L power:+5V #PWR0154
-U 1 1 5E97EB65
-P 6400 4650
-F 0 "#PWR0154" H 6400 4500 50  0001 C CNN
-F 1 "+5V" H 6415 4823 50  0000 C CNN
-F 2 "" H 6400 4650 50  0001 C CNN
-F 3 "" H 6400 4650 50  0001 C CNN
-	1    6400 4650
-	1    0    0    -1
-$EndComp
-Text Notes 6600 4550 0    79   ~ 0
-USB powered
-Wire Wire Line
-	6600 5150 7050 5150
-Wire Wire Line
-	7050 5050 7050 5150
-Connection ~ 7050 5150
-Wire Wire Line
-	7050 5150 7300 5150
 Connection ~ 1150 1000
 Wire Wire Line
@@
 	6500 1000 7000 1000
 $Comp
-L Device:D D8
+L gsvesc:SMMBD914LT3G D8
 U 1 1 5EA7F038
 P 7450 750
@@
 	3850 1000 4350 1000
 $Comp
-L Device:D D10
+L gsvesc:SMMBD914LT3G D10
 U 1 1 5EABE0CB
 P 4800 750
@@
 Connection ~ 5600 1000
 $Comp
-L Device:D D9
+L gsvesc:SMMBD914LT3G D9
 U 1 1 5EACAF3E
 P 2100 750
@@
 	1650 1000 1800 1000
 Connection ~ 2900 1000
+Wire Wire Line
+	6600 5150 7300 5150
 $EndSCHEMATC
