File: gsvesc_nrf.sch (KiCad schematic (older format))
At the start: 5 parts, among them J14 Conn_01x03, U16 EYSGJNZWY

Commit message: temp
Parts:
- J14: footprint Connector_JST:JST_SH_BM03B-SRSS-TB_1x03-1MP_P1.00mm_Vertical -> Connector_PinHeader_2.54mm:PinHeader_1x03_P2.54mm_Vertical
Changed lines of the file:
@@
 F 0 "J14" H 3270 4025 50  0000 C CNN
 F 1 "Conn_01x03" H 3270 4116 50  0000 C CNN
-F 2 "Connector_JST:JST_SH_BM03B-SRSS-TB_1x03-1MP_P1.00mm_Vertical" H 3350 4350 50  0001 C CNN
+F 2 "Connector_PinHeader_2.54mm:PinHeader_1x03_P2.54mm_Vertical" H 3350 4350 50  0001 C CNN
 F 3 "~" H 3350 4350 50  0001 C CNN
 	1    3350 4350
