File: gesc.kicad_pcb (KiCad board)
At the start: 4 copper layers, 111 x 111 mm, 164 parts, among them J1 Conn_01x06, J10 PHASE_C, J11 PHASE_B, J12 NTC, J13 T-Motor, J14 Conn_01x03, J15 EXT_OFF, J2 Conn_01x06, J3 Conn_01x06, J4 Conn_01x05, J5 Conn_01x03, J6 USB_B_Mini, J7 BAT+, J8 BAT-, J9 PHASE_A, Q1 BSC070N10NS5, Q2 BSC070N10NS5, Q3 BSC070N10NS5, Q4 BSC070N10NS5, Q5 BSC070N10NS5, Q6 BSC070N10NS5, U1 STM32F405RGTx, U10 LM5008MM, U11 SN74LVC1G66DBVR, U12 LM5107, U13 SN74LVC1G66DBVR, U14 AQY282S, U15 LM5107, U16 EYSGJNZWY, U17 LMR12010YMKE_NOPB, U2 SN74LVC1G66DBVR, U3 LM5107, U4 INA240A1, U5 INA240A1, U6 INA240A1, U7 SN74LVC1G66DBVR, U8 SN74LVC1G66DBVR, U9 SN74LVC1G66DBVR, Y1 X50328MSB2GI

Commit message: save
Parts:
- moved R36 24.7 mm to (61.0, 67.0), turned to 270 degrees
- moved J12 19.3 mm to (65.1, 67.0), turned to 270 degrees
Routing:
- net VCC: track 92.0 -> 110.6 mm
- net /MCU/ADC_TEMP: track 63.3 -> 68.3 mm
- net GND: track 116.6 -> 117.4 mm
- net /Driver/GL_B: track 24.8 -> 25.7 mm
- net /Driver/SH_B_R: track 35.9 -> 35.4 mm
