File: gesc.kicad_pcb (KiCad board)
At the start: 4 copper layers, 111 x 111 mm, 159 parts, among them J1 Conn_01x06, J10 PHASE_C, J11 PHASE_B, J13 T-Motor, J14 Conn_01x03, J15 EXT_OFF, J2 Conn_01x06, J3 Conn_01x06, J4 Conn_01x05, J5 Conn_01x03, J6 USB_B_Mini, J7 BAT+, J8 BAT-, J9 PHASE_A, Q1 BSC070N10NS5, Q2 BSC070N10NS5, Q3 BSC070N10NS5, Q4 BSC070N10NS5, Q5 BSC070N10NS5, Q6 BSC070N10NS5, U1 STM32F405RGTx, U10 LM5008MM, U11 SN74LVC1G66DBVR, U12 2ED2304S06F, U13 SN74LVC1G66DBVR, U14 AQY282S, U15 2ED2304S06F, U16 EYSGJNZWY, U17 TPS82140, U2 SN74LVC1G66DBVR, U3 2ED2304S06F, U4 INA240A1, U5 INA240A1, U6 INA240A1, U7 SN74LVC1G66DBVR, U8 SN74LVC1G66DBVR, U9 SN74LVC1G66DBVR, Y1 X50328MSB2GI

Commit message: Version rund platziert
Parts:
- removed R34: 330k, Resistor_SMD:R_0805_2012Metric
- removed R48: 110k, Resistor_SMD:R_0805_2012Metric
- added C50: 100n, Capacitor_SMD:C_0805_2012Metric, F.Cu at (94.9, 131.6)
- C33: value 3n30 -> 100n
- U17: value TPS82140 -> AMS1117-3.3; footprint Package_LGA:Texas_SIL0008D_MicroSiP-8-1EP_2.8x3mm_P0.65mm_EP1.1x1.9mm -> Package_TO_SOT_SMD:SOT-223-3_TabPin2
- moved C61 85.4 mm to (123.0, 58.8), turned to 60 degrees
- moved R25 81.8 mm to (128.0, 75.5), turned to 270 degrees
- moved C62 75.5 mm to (116.0, 70.5), turned to 240 degrees
- moved J11 74.9 mm to (86.3, 60.6)
- moved J10 73.7 mm to (131.7, 67.6), turned to 0 degrees
- moved Q3 73.1 mm to (132.3, 77.4), turned to 270 degrees
- moved R31 63.9 mm to (137.9, 73.1)
- moved C52 61.7 mm to (138.4, 79.6), turned to 0 degrees
- moved C43 61.6 mm to (138.4, 86.6), turned to 0 degrees
- moved C36 61.6 mm to (138.4, 83.1), turned to 0 degrees
- moved C58 61.4 mm to (124.6, 86.2), turned to 270 degrees
- moved C32 61.1 mm to (134.7, 83.7)
- moved U15 60.9 mm to (129.8, 84.6)
- moved C29 60.7 mm to (124.6, 82.6), turned to 90 degrees
- moved Q6 60.4 mm to (96.7, 55.7), turned to 180 degrees
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Connections:
- C33 pad 1: Net-(C33-Pad1) -> +12V
- U17 pad 1: (no net) -> GND
- U17 pad 2: +12V -> VCC
- U17 pad 3: GND -> +12V
Routing:
- net /Driver/SH_A: track 58.2 -> 14.2 mm, vias 39 -> 2
- net /POWER/PHASE_A: track 35.4 -> 1.30 mm, vias 51 -> 1
- net /Driver/GL_A: track 11.2 -> 0.00 mm, vias 2 -> 0
- net VBAT: track 92.0 -> 100.5 mm, vias 146 -> 73
- net /Driver/GH_A: track 6.84 -> 0.00 mm, vias 2 -> 0
- net /MCU/H1: track 40.5 -> 35.8 mm, vias 3 -> 2
- net /MCU/L1: track 47.0 -> 42.4 mm, vias 3 -> 2
- net Net-(R34-Pad2): track 3.98 -> 0.00 mm
- net Net-(C21-Pad1): track 2.93 -> 0.00 mm
- net VBUS: track 37.2 -> 39.9 mm
- net Net-(Q1-Pad4): track 2.57 -> 0.00 mm
- net /NRF/NRF_RX: track 91.8 -> 89.5 mm
- net /MCU/SERVO: track 68.7 -> 66.3 mm
- net /NRF/NRF_TX: track 89.3 -> 87.0 mm
- net GND: track 5.37 -> 3.12 mm, vias 93 -> 76
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- removed copper zone on F.Cu, net /Driver/SH_A
- removed copper zone on F.Cu, net /POWER/PHASE_A

Commit message: save
Parts:
- removed D5: B5819W, Diode_SMD:D_SOD-123
- moved J14 68.5 mm to (80.0, 118.7)
- moved C31 63.9 mm to (151.3, 93.8), turned to 180 degrees
- moved C17 63.3 mm to (151.3, 95.9), turned to 0 degrees
- moved C19 62.8 mm to (151.3, 98.1), turned to 0 degrees
- moved D6 61.0 mm to (150.3, 102.2), turned to 270 degrees
- moved C16 57.6 mm to (147.0, 95.3), turned to 180 degrees
- moved R23 57.3 mm to (147.7, 102.9), turned to 270 degrees
- moved U10 54.6 mm to (145.5, 99.0), turned to 0 degrees
- moved R16 54.4 mm to (145.7, 102.9), turned to 90 degrees
- moved R12 54.1 mm to (152.7, 102.6), turned to 270 degrees
- moved C23 51.4 mm to (143.6, 102.9), turned to 90 degrees
- moved D4 49.1 mm to (140.4, 93.7), turned to 0 degrees
- moved C20 48.8 mm to (141.1, 97.3), turned to 90 degrees
- moved R15 48.1 mm to (141.1, 101.0), turned to 270 degrees
- moved C26 47.8 mm to (141.0, 105.5), turned to 90 degrees
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Connections:
- J14 pad 1: GND -> Net-(J14-Pad1)
- J14 pad 2: Net-(J14-Pad2) -> GND
- J6 pad 1: VBUS -> (no net)
- U16 pad 16: Net-(J14-Pad2) -> Net-(J14-Pad3)
- U16 pad 17: Net-(J14-Pad3) -> Net-(J14-Pad1)
Routing:
- net GND: track 3.12 -> 92.9 mm, vias 76 -> 207
- net /Driver/SH_C: track 17.5 -> 107.0 mm, vias 2 -> 30
- net VBAT: track 100.5 -> 32.5 mm, vias 73 -> 141
- net /POWER/PHASE_C: track 3.53 -> 70.2 mm, vias 1 -> 27
- net /MCU/L3: track 26.6 -> 80.1 mm, vias 1 -> 2
- net /MCU/H3: track 23.5 -> 76.1 mm, vias 1 -> 2
- net /Driver/SH_B: track 23.4 -> 72.9 mm, vias 2 -> 30
- net /NRF/NRF_RX: track 89.5 -> 48.4 mm
- net VBUS: track 39.9 -> 0.00 mm, vias 1 -> 0
- net /NRF/NRF_TX: track 87.0 -> 47.1 mm
- net /Driver/SH_A: track 14.2 -> 53.2 mm, vias 2 -> 30
- net /MCU/H2: track 25.5 -> 59.4 mm, vias 1 -> 2
- net /POWER/PHASE_B: track 9.98 -> 42.9 mm, vias 1 -> 27
- net /MCU/L2: track 29.7 -> 59.4 mm, vias 1 -> 2
- net Net-(J14-Pad2): track 25.5 -> 0.00 mm, vias 1 -> 0
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- added copper zone on B.Cu, net /Driver/SH_A
- added copper zone on F.Cu, net /Driver/SH_A
- added copper zone on B.Cu, net /Driver/SH_B
- added copper zone on F.Cu, net /Driver/SH_B
- added copper zone on B.Cu, net /Driver/SH_C
- added copper zone on F.Cu, net /Driver/SH_C
- added copper zone on B.Cu, net /POWER/PHASE_A
- added copper zone on F.Cu, net /POWER/PHASE_A
- added copper zone on B.Cu, net /POWER/PHASE_B
- added copper zone on F.Cu, net /POWER/PHASE_B
- added copper zone on B.Cu, net /POWER/PHASE_C
- added copper zone on F.Cu, net /POWER/PHASE_C
- added copper zone on B.Cu, net VBAT

Commit message: save
Parts:
- added TP1: Antenna, TestPoint:TestPoint_Pad_D2.0mm, F.Cu at (116.8, 149.2)
- added U18: RFM95W-868S2, gesc:XCVR_RFM95W-868S2, F.Cu at (116.6, 137.6)
- Q1, Q2, Q3, Q4, Q5, Q6: value BSC070N10NS5 -> TPH2R608NH; footprint Package_TO_SOT_SMD:TDSON-8-1 -> gesc:TRANS_TPHR8504PL-3PIN
- moved Q4 0.26 mm to (135.8, 67.5)
- moved Q3 0.22 mm to (124.9, 67.2)
- moved Q6 0.12 mm to (91.5, 56.6)
- moved Q5 0.10 mm to (92.1, 68.0)
- moved Q1 0.07 mm to (64.3, 77.1)
Connections:
- net /NRF/NRF_RX renamed /RF Module/NRF_RX_MISO
- net /NRF/NRF_TX renamed /RF Module/NRF_TX_SCK
- Q1 pad 1: /Driver/SH_A -> VBAT
- Q1 pad 2: /Driver/SH_A -> Net-(Q1-Pad2)
- Q2 pad 1: GND -> /Driver/SH_A
- Q2 pad 2: GND -> Net-(Q2-Pad2)
- Q3 pad 1: /Driver/SH_C -> VBAT
- Q3 pad 2: /Driver/SH_C -> Net-(Q3-Pad2)
- Q4 pad 1: GND -> /Driver/SH_C
- Q4 pad 2: GND -> Net-(Q4-Pad2)
- Q5 pad 1: /Driver/SH_B -> VBAT
- Q5 pad 2: /Driver/SH_B -> Net-(Q5-Pad2)
- Q6 pad 1: GND -> /Driver/SH_B
- Q6 pad 2: GND -> Net-(Q6-Pad2)
- R25 pad 1: Net-(Q3-Pad4) -> Net-(Q3-Pad2)
- R26 pad 1: Net-(Q4-Pad4) -> Net-(Q4-Pad2)
- R28 pad 1: Net-(Q1-Pad4) -> Net-(Q1-Pad2)
- R32 pad 1: Net-(Q2-Pad4) -> Net-(Q2-Pad2)
- R42 pad 1: Net-(Q5-Pad4) -> Net-(Q5-Pad2)
- R43 pad 1: Net-(Q6-Pad4) -> Net-(Q6-Pad2)
- U1 pad 33: (no net) -> /RF Module/DIO0
- U1 pad 50: (no net) -> /RF Module/NSS
- U1 pad 53: (no net) -> /RF Module/MOSI
- U1 pad 58: (no net) -> /MCU/PB6
Routing:
- net /RF Module/MOSI: track 0.00 -> 87.1 mm, vias 0 -> 3
- net /RF Module/NSS: track 0.00 -> 82.9 mm, vias 0 -> 4
- net /MCU/PB6: track 0.00 -> 80.9 mm, vias 0 -> 3
- net /RF Module/DIO0: track 0.00 -> 78.4 mm, vias 0 -> 3
- net /RF Module/NRF_RX_MISO: track 48.4 -> 88.1 mm, vias 3 -> 4
- net /RF Module/NRF_TX_SCK: track 47.1 -> 81.3 mm, vias 3 -> 4
- net Net-(TP1-Pad1): track 0.00 -> 10.7 mm
- net /MCU/I2C1_SDA: track 38.6 -> 35.5 mm
- net Net-(Q3-Pad4): track 2.35 -> 0.00 mm
- net Net-(Q3-Pad2): track 0.00 -> 2.35 mm
- net Net-(Q5-Pad4): track 2.28 -> 0.00 mm
- net Net-(Q5-Pad2): track 0.00 -> 2.28 mm
- net Net-(Q1-Pad4): track 2.23 -> 0.00 mm
- net Net-(Q1-Pad2): track 0.00 -> 2.23 mm
- net Net-(Q4-Pad4): track 2.20 -> 0.00 mm
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Other:
- net class Default: trace_width 0.15 -> 0.2

Commit message: save
Parts:
- removed R44: 2k10, Resistor_SMD:R_0805_2012Metric
Connections:
- net /RF Module/DIO0 renamed /HF Module/DIO0
- U1 pad 28: (no net) -> /MCU/PB2
- U1 pad 50: /RF Module/NSS -> (no net)
- U1 pad 51: /RF Module/NRF_TX_SCK -> /HF Module/NRF_TX_SCK
- U1 pad 52: /RF Module/NRF_RX_MISO -> /HF Module/NRF_RX_MISO
- U1 pad 53: /RF Module/MOSI -> (no net)
- U1 pad 55: (no net) -> /HF Module/NSS
- U1 pad 56: (no net) -> /HF Module/MOSI
- U1 pad 57: (no net) -> /HF Module/MISO
- U16 pad 21: /RF Module/NRF_TX_SCK -> /HF Module/NRF_TX_SCK
- U16 pad 22: /RF Module/NRF_RX_MISO -> /HF Module/NRF_RX_MISO
- U18 pad 2: /RF Module/NRF_RX_MISO -> /HF Module/MISO
- U18 pad 3: /RF Module/MOSI -> /HF Module/MOSI
- U18 pad 4: /RF Module/NRF_TX_SCK -> /MCU/PB6
- U18 pad 5: /RF Module/NSS -> /HF Module/NSS
- U18 pad 6: /MCU/PB6 -> /MCU/PB2
Routing:
- net /RF Module/NRF_RX_MISO: track 88.1 -> 0.00 mm, vias 4 -> 0
- net /RF Module/MOSI: track 87.1 -> 0.00 mm, vias 3 -> 0
- net /HF Module/MOSI: track 0.00 -> 87.0 mm, vias 0 -> 3
- net /HF Module/NSS: track 0.00 -> 86.7 mm, vias 0 -> 4
- net /HF Module/MISO: track 0.00 -> 86.1 mm, vias 0 -> 3
- net /RF Module/NSS: track 82.9 -> 0.00 mm, vias 4 -> 0
- net /RF Module/NRF_TX_SCK: track 81.3 -> 0.00 mm, vias 4 -> 0
- net /MCU/PB2: track 0.00 -> 67.0 mm, vias 0 -> 3
- net /HF Module/NRF_RX_MISO: track 0.00 -> 48.8 mm, vias 0 -> 3
- net /HF Module/NRF_TX_SCK: track 0.00 -> 47.2 mm, vias 0 -> 3
- net /MCU/PB6: track 80.9 -> 85.4 mm
- net /MCU/MISO_ADC_EXT2: track 59.4 -> 58.6 mm
Other:
- rule pad_to_mask_clearance: 0.051 -> 0
