File: gesc.sch (KiCad schematic (older format))
At the start: 38 parts, among them J1 Conn_01x06, J13 T-Motor, J15 EXT_OFF, J2 Conn_01x06, J3 Conn_01x06, J4 Conn_01x05, J5 Conn_01x03, J6 USB_B_Mini, J7 BAT+, J8 BAT-

Commit message: save
Connections:
- no-connect marks 6 -> 5
Other:
- moved on the sheet: D1, D2, D3, R10, R11, R9
Changed lines of the file:
@@
 L Device:R R9
 U 1 1 5BEBF9DC
-P 6150 5800
-F 0 "R9" V 6100 5950 50  0000 C CNN
-F 1 "1k00" V 6150 5800 50  0000 C CNN
-F 2 "Resistor_SMD:R_0805_2012Metric" V 6080 5800 50  0001 C CNN
-F 3 "~" H 6150 5800 50  0001 C CNN
-	1    6150 5800
+P 6150 6150
+F 0 "R9" V 6100 6300 50  0000 C CNN
+F 1 "1k00" V 6150 6150 50  0000 C CNN
+F 2 "Resistor_SMD:R_0805_2012Metric" V 6080 6150 50  0001 C CNN
+F 3 "~" H 6150 6150 50  0001 C CNN
+	1    6150 6150
 	0    1    1    0
 $EndComp
@@
 L Device:R R10
 U 1 1 5BEBFA63
-P 6150 5950
-F 0 "R10" V 6100 6100 50  0000 C CNN
-F 1 "221r" V 6150 5950 50  0000 C CNN
-F 2 "Resistor_SMD:R_0805_2012Metric" V 6080 5950 50  0001 C CNN
-F 3 "~" H 6150 5950 50  0001 C CNN
-	1    6150 5950
+P 6150 6300
+F 0 "R10" V 6100 6450 50  0000 C CNN
+F 1 "221r" V 6150 6300 50  0000 C CNN
+F 2 "Resistor_SMD:R_0805_2012Metric" V 6080 6300 50  0001 C CNN
+F 3 "~" H 6150 6300 50  0001 C CNN
+	1    6150 6300
 	0    1    1    0
 $EndComp
@@
 L Device:R R11
 U 1 1 5BEBFADA
-P 6150 6100
-F 0 "R11" V 6100 6250 50  0000 C CNN
-F 1 "221r" V 6150 6100 50  0000 C CNN
-F 2 "Resistor_SMD:R_0805_2012Metric" V 6080 6100 50  0001 C CNN
-F 3 "~" H 6150 6100 50  0001 C CNN
-	1    6150 6100
-	0    1    1    0
-$EndComp
-Wire Wire Line
-	4600 6100 5350 6100
-Wire Wire Line
-	4600 6000 5150 6000
-Wire Wire Line
-	5150 6000 5150 5950
-Wire Wire Line
-	5150 5950 5350 5950
-Wire Wire Line
-	5250 5800 5350 5800
-Wire Wire Line
-	6300 5800 6500 5800
-Wire Wire Line
-	6500 5800 6500 5950
-Wire Wire Line
-	6300 6100 6500 6100
-Connection ~ 6500 6100
-Wire Wire Line
-	6500 6100 6500 6350
-Wire Wire Line
-	6300 5950 6500 5950
-Connection ~ 6500 5950
-Wire Wire Line
-	6500 5950 6500 6100
+P 6150 6450
+F 0 "R11" V 6100 6600 50  0000 C CNN
+F 1 "221r" V 6150 6450 50  0000 C CNN
+F 2 "Resistor_SMD:R_0805_2012Metric" V 6080 6450 50  0001 C CNN
+F 3 "~" H 6150 6450 50  0001 C CNN
+	1    6150 6450
+	0    1    1    0
+$EndComp
+Wire Wire Line
+	4600 6450 5350 6450
+Wire Wire Line
+	4600 6350 5150 6350
+Wire Wire Line
+	5150 6350 5150 6300
+Wire Wire Line
+	5150 6300 5350 6300
+Wire Wire Line
+	5250 6150 5350 6150
+Wire Wire Line
+	6300 6150 6500 6150
+Wire Wire Line
+	6500 6150 6500 6300
+Wire Wire Line
+	6300 6450 6500 6450
+Connection ~ 6500 6450
+Wire Wire Line
+	6500 6450 6500 6700
+Wire Wire Line
+	6300 6300 6500 6300
+Connection ~ 6500 6300
+Wire Wire Line
+	6500 6300 6500 6450
 $Comp
 L power:VCC #PWR016
 U 1 1 5BEC80D8
-P 5250 5800
-F 0 "#PWR016" H 5250 5650 50  0001 C CNN
-F 1 "VCC" V 5268 5927 50  0000 L CNN
-F 2 "" H 5250 5800 50  0001 C CNN
-F 3 "" H 5250 5800 50  0001 C CNN
-	1    5250 5800
+P 5250 6150
+F 0 "#PWR016" H 5250 6000 50  0001 C CNN
+F 1 "VCC" V 5268 6277 50  0000 L CNN
+F 2 "" H 5250 6150 50  0001 C CNN
+F 3 "" H 5250 6150 50  0001 C CNN
+	1    5250 6150
 	0    -1   -1   0
 $EndComp
@@
 L Device:LED D1
 U 1 1 5BEC97C2
-P 5500 5800
-F 0 "D1" H 5400 5850 50  0000 C CNN
-F 1 "BLUE" H 5650 5850 50  0000 C CNN
-F 2 "LED_SMD:LED_0805_2012Metric" H 5500 5800 50  0001 C CNN
-F 3 "~" H 5500 5800 50  0001 C CNN
-	1    5500 5800
+P 5500 6150
+F 0 "D1" H 5400 6200 50  0000 C CNN
+F 1 "BLUE" H 5650 6200 50  0000 C CNN
+F 2 "LED_SMD:LED_0805_2012Metric" H 5500 6150 50  0001 C CNN
+F 3 "~" H 5500 6150 50  0001 C CNN
+	1    5500 6150
 	-1   0    0    1
 $EndComp
 Wire Wire Line
-	5650 5800 6000 5800
+	5650 6150 6000 6150
 $Comp
 L Device:LED D3
 U 1 1 5BEC9894
-P 5500 6100
-F 0 "D3" H 5400 6150 50  0000 C CNN
-F 1 "GREEN" H 5700 6150 50  0000 C CNN
-F 2 "LED_SMD:LED_0805_2012Metric" H 5500 6100 50  0001 C CNN
-F 3 "~" H 5500 6100 50  0001 C CNN
-	1    5500 6100
+P 5500 6450
+F 0 "D3" H 5400 6500 50  0000 C CNN
+F 1 "GREEN" H 5700 6500 50  0000 C CNN
+F 2 "LED_SMD:LED_0805_2012Metric" H 5500 6450 50  0001 C CNN
+F 3 "~" H 5500 6450 50  0001 C CNN
+	1    5500 6450
 	-1   0    0    1
 $EndComp
 Wire Wire Line
-	5650 6100 6000 6100
+	5650 6450 6000 6450
 $Comp
 L Device:LED D2
 U 1 1 5BECC59F
-P 5500 5950
-F 0 "D2" H 5400 6000 50  0000 C CNN
-F 1 "RED" H 5650 6000 50  0000 C CNN
-F 2 "LED_SMD:LED_0805_2012Metric" H 5500 5950 50  0001 C CNN
-F 3 "~" H 5500 5950 50  0001 C CNN
-	1    5500 5950
+P 5500 6300
+F 0 "D2" H 5400 6350 50  0000 C CNN
+F 1 "RED" H 5650 6350 50  0000 C CNN
+F 2 "LED_SMD:LED_0805_2012Metric" H 5500 6300 50  0001 C CNN
+F 3 "~" H 5500 6300 50  0001 C CNN
+	1    5500 6300
 	-1   0    0    1
 $EndComp
 Wire Wire Line
-	5650 5950 6000 5950
+	5650 6300 6000 6300
 $Comp
 L power:GND #PWR017
 U 1 1 5BECCAF3
-P 6500 6350
-F 0 "#PWR017" H 6500 6100 50  0001 C CNN
-F 1 "GND" H 6505 6177 50  0000 C CNN
-F 2 "" H 6500 6350 50  0001 C CNN
-F 3 "" H 6500 6350 50  0001 C CNN
-	1    6500 6350
+P 6500 6700
+F 0 "#PWR017" H 6500 6450 50  0001 C CNN
+F 1 "GND" H 6505 6527 50  0000 C CNN
+F 2 "" H 6500 6700 50  0001 C CNN
+F 3 "" H 6500 6700 50  0001 C CNN
+	1    6500 6700
 	1    0    0    -1
 $EndComp
 $Sheet
-S 5200 4950 900  550
+S 5200 5200 900  650
 U 5BECFBE3
-F0 "NRF" 50
+F0 "RF Module" 50
 F1 "gesc_nrf.sch" 50
-F2 "NRF_TX" I L 5200 5300 50
-F3 "NRF_RX" I L 5200 5400 50
-F4 "GPIO1" I L 5200 5000 50
-F5 "GPIO2" I L 5200 5100 50
-F6 "GPIO3" I L 5200 5200 50
+F2 "NRF_TX_SCK" I L 5200 5550 50
+F3 "NRF_RX_MISO" I L 5200 5650 50
+F4 "MOSI" I L 5200 5450 50
+F5 "NSS" I L 5200 5350 50
+F6 "RESET" I L 5200 5250 50
+F7 "DIO0" I L 5200 5750 50
 $EndSheet
 Wire Wire Line
@@
 $EndComp
 NoConn ~ 1900 1900
-NoConn ~ 4600 4300
-NoConn ~ 4600 4400
 $Comp
 L power:PWR_FLAG #FLG0102
@@
 	2350 1700 3250 1700
 Wire Wire Line
-	4600 5300 5200 5300
-Wire Wire Line
-	4600 5400 5200 5400
+	4600 5550 5200 5550
+Wire Wire Line
+	4600 5650 5200 5650
 Wire Wire Line
 	4600 3700 7550 3700
 Wire Wire Line
-	4600 5000 5200 5000
-Wire Wire Line
-	4600 5100 5200 5100
-Wire Wire Line
-	4600 5200 5200 5200
+	4600 5250 5200 5250
+Wire Wire Line
+	4600 5350 5200 5350
+Wire Wire Line
+	4600 5450 5200 5450
 $Comp
 L Mechanical:MountingHole H1
@@
 	1    0    0    -1
 $EndComp
-Wire Wire Line
-	1700 5300 3250 5300
-$Sheet
-S 3250 1450 1350 5200
-U 5BE81C34
-F0 "MCU" 50
-F1 "gesc_uc.sch" 50
-F2 "USB_D+" B L 3250 1700 50
-F3 "USB_D-" B L 3250 1800 50
-F4 "TEMP_MOTOR" I L 3250 3350 50
-F5 "TX_SCL_MOSI" O L 3250 4150 50
-F6 "MISO_ADC_EXT2" I L 3250 4250 50
-F7 "SCK_ADC_EXT" I L 3250 4350 50
-F8 "RX_SDA_NSS" B L 3250 4450 50
-F9 "HALL_TRIG" I L 3250 5000 50
-F10 "HALL_ROT_A" I L 3250 5100 50
-F11 "HALL_ROT_B" I L 3250 5200 50
-F12 "SWCLK" I L 3250 6250 50
-F13 "NRST" I L 3250 5950 50
-F14 "SWDIO" B L 3250 6050 50
-F15 "SERVO" O L 3250 6500 50
-F16 "LED_RED" O R 4600 6000 50
-F17 "LED_GREEN" O R 4600 6100 50
-F18 "H1" O R 4600 1550 50
-F19 "H2" O R 4600 1650 50
-F20 "H3" O R 4600 1750 50
-F21 "L1" O R 4600 1850 50
-F22 "L2" O R 4600 1950 50
-F23 "L3" O R 4600 2050 50
-F24 "VOLTAGE_1" I R 4600 3000 50
-F25 "VOLTAGE_2" I R 4600 3100 50
-F26 "VOLTAGE_3" I R 4600 3200 50
-F27 "AN_IN" I R 4600 3300 50
-F28 "CURRENT_1" I R 4600 3800 50
-F29 "CURRENT_2" I R 4600 3900 50
-F30 "CURRENT_3" I R 4600 4000 50
-F31 "ADC_TEMP" I R 4600 4100 50
-F32 "HALL_1" I L 3250 3050 50
-F33 "HALL_2" I L 3250 3150 50
-F34 "HALL_3" I L 3250 3250 50
-F35 "PC5" I L 3250 5300 50
-F36 "PA15" I R 4600 4300 50
-F37 "PB2" I R 4600 5000 50
-F38 "PB3" I R 4600 5100 50
-F39 "PB4" I R 4600 5200 50
-F40 "P_UART_TX" I R 4600 5300 50
-F41 "P_UART_RX" I R 4600 5400 50
-F42 "PB12" I R 4600 4400 50
-F43 "CURR_FILTER_ON" O R 4600 3700 50
-F44 "SENS_FILTER_ON" I R 4600 2800 50
-F45 "I2C1_SCL" I L 3250 4700 50
-F46 "I2C1_SDA" I L 3250 4800 50
-F47 "PB5" I R 4600 2250 50
-F48 "PB6" I R 4600 2350 50
-F49 "PC12" I R 4600 2450 50
-$EndSheet
 $Sheet
 S 5450 1450 1050 1950
@@
 	1    0    0    -1
 $EndComp
-NoConn ~ 4600 2250
-NoConn ~ 4600 2350
-NoConn ~ 4600 2450
 $Comp
 L Connector_Generic:Conn_01x06 J15
@@
 Wire Wire Line
 	6500 1550 6950 1550
+Wire Wire Line
+	1700 5300 3250 5300
+Wire Wire Line
+	4600 5750 5200 5750
+$Sheet
+S 3250 1450 1350 5200
+U 5BE81C34
+F0 "MCU" 50
+F1 "gesc_uc.sch" 50
+F2 "USB_D+" B L 3250 1700 50
+F3 "USB_D-" B L 3250 1800 50
+F4 "TEMP_MOTOR" I L 3250 3350 50
+F5 "TX_SCL_MOSI" O L 3250 4150 50
+F6 "MISO_ADC_EXT2" I L 3250 4250 50
+F7 "SCK_ADC_EXT" I L 3250 4350 50
+F8 "RX_SDA_NSS" B L 3250 4450 50
+F9 "HALL_TRIG" I L 3250 5000 50
+F10 "HALL_ROT_A" I L 3250 5100 50
+F11 "HALL_ROT_B" I L 3250 5200 50
+F12 "SWCLK" I L 3250 6250 50
+F13 "NRST" I L 3250 5950 50
+F14 "SWDIO" B L 3250 6050 50
+F15 "SERVO" O L 3250 6500 50
+F16 "LED_RED" O R 4600 6350 50
+F17 "LED_GREEN" O R 4600 6450 50
+F18 "H1" O R 4600 1550 50
+F19 "H2" O R 4600 1650 50
+F20 "H3" O R 4600 1750 50
+F21 "L1" O R 4600 1850 50
+F22 "L2" O R 4600 1950 50
+F23 "L3" O R 4600 2050 50
+F24 "VOLTAGE_1" I R 4600 3000 50
+F25 "VOLTAGE_2" I R 4600 3100 50
+F26 "VOLTAGE_3" I R 4600 3200 50
+F27 "AN_IN" I R 4600 3300 50
+F28 "CURRENT_1" I R 4600 3800 50
+F29 "CURRENT_2" I R 4600 3900 50
+F30 "CURRENT_3" I R 4600 4000 50
+F31 "ADC_TEMP" I R 4600 4100 50
+F32 "HALL_1" I L 3250 3050 50
+F33 "HALL_2" I L 3250 3150 50
+F34 "HALL_3" I L 3250 3250 50
+F35 "PC5" I L 3250 5300 50
+F36 "PB4" I R 4600 4550 50
+F37 "CURR_FILTER_ON" O R 4600 3700 50
+F38 "SENS_FILTER_ON" I R 4600 2800 50
+F39 "I2C1_SCL" I L 3250 4700 50
+F40 "I2C1_SDA" I L 3250 4800 50
+F41 "PB5" I R 4600 4650 50
+F42 "PB6" I R 4600 5250 50
+F43 "SPI3_NSS" I R 4600 5350 50
+F44 "P_UART_TX_SCK" I R 4600 5550 50
+F45 "P_UART_RX_MISO" I R 4600 5650 50
+F46 "SPI3_MOSI" I R 4600 5450 50
+F47 "PB2" I R 4600 4350 50
+F48 "PB12" I R 4600 5750 50
+F49 "PB3" I R 4600 4450 50
+$EndSheet
+NoConn ~ 4600 4350
+NoConn ~ 4600 4450
+NoConn ~ 4600 4550
+NoConn ~ 4600 4650
 $EndSCHEMATC
