File: gesc.sch (KiCad schematic (older format))
At the start: 38 parts, among them J1 Conn_01x06, J13 T-Motor, J15 EXT_OFF, J2 Conn_01x06, J3 Conn_01x06, J4 Conn_01x05, J5 Conn_01x03, J6 USB_B_Mini, J7 BAT+, J8 BAT-

Commit message: save
Parts:
- J6: symbol Connector:USB_B_Mini -> gesc-rescue:USB_B_Mini-Connector
Connections:
- no-connect marks 5 -> 1
Changed lines of the file:
@@
 Overview and Connector
 $Comp
-L Connector:USB_B_Mini J6
+L gesc-rescue:USB_B_Mini-Connector J6
 U 1 1 5BE8753D
 P 1600 1700
@@
 $EndComp
 $Sheet
-S 5200 5200 900  650
+S 5200 5100 1300 800
 U 5BECFBE3
-F0 "RF Module" 50
+F0 "HF Module" 50
 F1 "gesc_nrf.sch" 50
-F2 "NRF_TX_SCK" I L 5200 5550 50
-F3 "NRF_RX_MISO" I L 5200 5650 50
-F4 "MOSI" I L 5200 5450 50
-F5 "NSS" I L 5200 5350 50
-F6 "RESET" I L 5200 5250 50
-F7 "DIO0" I L 5200 5750 50
+F2 "NRF_TX_SCK" I L 5200 5750 50
+F3 "NRF_RX_MISO" I L 5200 5850 50
+F4 "MOSI" I L 5200 5350 50
+F5 "NSS" I L 5200 5250 50
+F6 "RESET" I L 5200 5150 50
+F7 "SCK" I L 5200 5550 50
+F8 "MISO" I L 5200 5450 50
+F9 "DIO0" I L 5200 5650 50
 $EndSheet
 Wire Wire Line
@@
 	2350 1700 3250 1700
 Wire Wire Line
-	4600 5550 5200 5550
-Wire Wire Line
-	4600 5650 5200 5650
+	4600 5750 5200 5750
+Wire Wire Line
+	4600 5850 5200 5850
 Wire Wire Line
 	4600 3700 7550 3700
 Wire Wire Line
+	4600 5150 5200 5150
+Wire Wire Line
 	4600 5250 5200 5250
 Wire Wire Line
 	4600 5350 5200 5350
-Wire Wire Line
-	4600 5450 5200 5450
 $Comp
 L Mechanical:MountingHole H1
@@
 Wire Wire Line
 	1700 5300 3250 5300
-Wire Wire Line
-	4600 5750 5200 5750
 $Sheet
 S 3250 1450 1350 5200
@@
 F34 "HALL_3" I L 3250 3250 50
 F35 "PC5" I L 3250 5300 50
-F36 "PB4" I R 4600 4550 50
+F36 "PB4" I R 4600 5350 50
 F37 "CURR_FILTER_ON" O R 4600 3700 50
 F38 "SENS_FILTER_ON" I R 4600 2800 50
 F39 "I2C1_SCL" I L 3250 4700 50
 F40 "I2C1_SDA" I L 3250 4800 50
-F41 "PB5" I R 4600 4650 50
-F42 "PB6" I R 4600 5250 50
-F43 "SPI3_NSS" I R 4600 5350 50
-F44 "P_UART_TX_SCK" I R 4600 5550 50
-F45 "P_UART_RX_MISO" I R 4600 5650 50
-F46 "SPI3_MOSI" I R 4600 5450 50
-F47 "PB2" I R 4600 4350 50
-F48 "PB12" I R 4600 5750 50
-F49 "PB3" I R 4600 4450 50
+F41 "PB5" I R 4600 5450 50
+F42 "PB6" I R 4600 5550 50
+F43 "P_UART_TX_SCK" I R 4600 5750 50
+F44 "P_UART_RX_MISO" I R 4600 5850 50
+F45 "PB2" I R 4600 5150 50
+F46 "PB12" I R 4600 5650 50
+F47 "PB3" I R 4600 5250 50
 $EndSheet
-NoConn ~ 4600 4350
-NoConn ~ 4600 4450
-NoConn ~ 4600 4550
-NoConn ~ 4600 4650
+Wire Wire Line
+	4600 5450 5200 5450
+Wire Wire Line
+	4600 5550 5200 5550
+Wire Wire Line
+	4600 5650 5200 5650
 $EndSCHEMATC

Commit message: V7 PCB order
Connections:
- net USB_5V: now reaches J6.1 (VBUS)
Changed lines of the file:
@@
 Wire Wire Line
 	4600 5650 5200 5650
+Wire Wire Line
+	1900 1500 2150 1500
+Text GLabel 2150 1500 2    50   Input ~ 0
+USB_5V
 $EndSCHEMATC
