File: gesc_pwr.sch (KiCad schematic (older format))
At the start: 48 parts, among them J10 PHASE_C, J11 PHASE_B, J9 PHASE_A, Q1 BSC070N10NS5, Q2 BSC070N10NS5, Q3 BSC070N10NS5, Q4 BSC070N10NS5, Q5 BSC070N10NS5, Q6 BSC070N10NS5, U4 INA240A1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

Commit message: save
Parts:
- removed Q1, Q2, Q3, Q4, Q5, Q6: BSC070N10NS5, Package_TO_SOT_SMD:TDSON-8-1, symbol Transistor_FET:BSC070N10NS5
- added Q1, Q2, Q3, Q4, Q5, Q6: TPH2R608NH, gesc:TRANS_TPHR8504PL-3PIN, symbol gesc:TPH2R608NH
Connections:
- net GND: now also Q2.3 (S), Q4.3 (S), Q6.3 (S)
- net SH_A: now also Q1.3 (S), Q2.1 (D)
- net SH_B: now also Q5.3 (S), Q6.1 (D)
- net SH_C: now also Q3.3 (S), Q4.1 (D)
- net VBAT: now also Q1.1 (D), Q3.1 (D), Q5.1 (D)
- net at R26.1: now also Q4.2 (G)
- net at R25.1: now also Q3.2 (G)
- net at R43.1: now also Q6.2 (G)
- net at R42.1: now also Q5.2 (G)
- net at R32.1: now also Q2.2 (G)
- net at R28.1: now also Q1.2 (G)
Changed lines of the file:
@@
 $Descr A4 11693 8268
 encoding utf-8
-Sheet 5 5
+Sheet 4 5
 Title "GESC - DC Motor Controler"
 Date "2020-04-09"
@@
 	2800 6200 2800 6900
 $Comp
-L Transistor_FET:BSC070N10NS5 Q3
-U 1 1 601290B0
-P 1650 1300
-F 0 "Q3" H 1854 1346 50  0000 L CNN
-F 1 "BSC070N10NS5" H 1854 1255 50  0000 L CNN
-F 2 "Package_TO_SOT_SMD:TDSON-8-1" H 1850 1225 50  0001 L CIN
-F 3 "http://www.infineon.com/dgdl/Infineon-BSC070N10NS5-DS-v02_01-EN.pdf?fileId=5546d4624a0bf290014a0fc62d9d6b3c" V 1650 1300 50  0001 L CNN
-	1    1650 1300
-	1    0    0    -1
-$EndComp
-$Comp
-L Transistor_FET:BSC070N10NS5 Q4
-U 1 1 60131502
-P 1650 1950
-F 0 "Q4" H 1854 1996 50  0000 L CNN
-F 1 "BSC070N10NS5" H 1854 1905 50  0000 L CNN
-F 2 "Package_TO_SOT_SMD:TDSON-8-1" H 1850 1875 50  0001 L CIN
-F 3 "http://www.infineon.com/dgdl/Infineon-BSC070N10NS5-DS-v02_01-EN.pdf?fileId=5546d4624a0bf290014a0fc62d9d6b3c" V 1650 1950 50  0001 L CNN
-	1    1650 1950
-	1    0    0    -1
-$EndComp
-$Comp
-L Transistor_FET:BSC070N10NS5 Q5
-U 1 1 60136E0E
-P 1650 3500
-F 0 "Q5" H 1854 3546 50  0000 L CNN
-F 1 "BSC070N10NS5" H 1854 3455 50  0000 L CNN
-F 2 "Package_TO_SOT_SMD:TDSON-8-1" H 1850 3425 50  0001 L CIN
-F 3 "http://www.infineon.com/dgdl/Infineon-BSC070N10NS5-DS-v02_01-EN.pdf?fileId=5546d4624a0bf290014a0fc62d9d6b3c" V 1650 3500 50  0001 L CNN
-	1    1650 3500
-	1    0    0    -1
-$EndComp
-$Comp
-L Transistor_FET:BSC070N10NS5 Q6
-U 1 1 601394AD
-P 1650 4150
-F 0 "Q6" H 1854 4196 50  0000 L CNN
-F 1 "BSC070N10NS5" H 1854 4105 50  0000 L CNN
-F 2 "Package_TO_SOT_SMD:TDSON-8-1" H 1850 4075 50  0001 L CIN
-F 3 "http://www.infineon.com/dgdl/Infineon-BSC070N10NS5-DS-v02_01-EN.pdf?fileId=5546d4624a0bf290014a0fc62d9d6b3c" V 1650 4150 50  0001 L CNN
-	1    1650 4150
-	1    0    0    -1
-$EndComp
-$Comp
-L Transistor_FET:BSC070N10NS5 Q1
-U 1 1 6013C3DE
-P 1600 5950
-F 0 "Q1" H 1804 5996 50  0000 L CNN
-F 1 "BSC070N10NS5" H 1804 5905 50  0000 L CNN
-F 2 "Package_TO_SOT_SMD:TDSON-8-1" H 1800 5875 50  0001 L CIN
-F 3 "http://www.infineon.com/dgdl/Infineon-BSC070N10NS5-DS-v02_01-EN.pdf?fileId=5546d4624a0bf290014a0fc62d9d6b3c" V 1600 5950 50  0001 L CNN
-	1    1600 5950
-	1    0    0    -1
-$EndComp
-$Comp
-L Transistor_FET:BSC070N10NS5 Q2
-U 1 1 6013F03F
-P 1600 6600
-F 0 "Q2" H 1804 6646 50  0000 L CNN
-F 1 "BSC070N10NS5" H 1804 6555 50  0000 L CNN
-F 2 "Package_TO_SOT_SMD:TDSON-8-1" H 1800 6525 50  0001 L CIN
-F 3 "http://www.infineon.com/dgdl/Infineon-BSC070N10NS5-DS-v02_01-EN.pdf?fileId=5546d4624a0bf290014a0fc62d9d6b3c" V 1600 6600 50  0001 L CNN
-	1    1600 6600
-	1    0    0    -1
-$EndComp
-$Comp
 L Device:R R47
 U 1 1 606B4BF8
@@
 Wire Wire Line
 	10050 1100 10050 1250
+$Comp
+L gesc:TPH2R608NH Q3
+U 1 1 604A2739
+P 1650 1300
+F 0 "Q3" H 1856 1346 50  0000 L CNN
+F 1 "TPH2R608NH" H 1856 1255 50  0000 L CNN
+F 2 "gesc:TRANS_TPHR8504PL-3PIN" H 1650 1300 50  0001 C CIN
+F 3 "" H 1650 1300 50  0001 L CNN
+F 4 "TPH2R608NH" H 2300 2300 236 0001 C CNN "Partnumber"
+F 5 "C146377" H 1950 2000 236 0001 C CNN "LCSC"
+	1    1650 1300
+	1    0    0    -1
+$EndComp
+$Comp
+L gesc:TPH2R608NH Q4
+U 1 1 604AB583
+P 1650 1950
+F 0 "Q4" H 1856 1996 50  0000 L CNN
+F 1 "TPH2R608NH" H 1856 1905 50  0000 L CNN
+F 2 "gesc:TRANS_TPHR8504PL-3PIN" H 1650 1950 50  0001 C CIN
+F 3 "" H 1650 1950 50  0001 L CNN
+F 4 "TPH2R608NH" H 2300 2950 236 0001 C CNN "Partnumber"
+F 5 "C146377" H 1950 2650 236 0001 C CNN "LCSC"
+	1    1650 1950
+	1    0    0    -1
+$EndComp
+$Comp
+L gesc:TPH2R608NH Q5
+U 1 1 604B4ADD
+P 1650 3500
+F 0 "Q5" H 1856 3546 50  0000 L CNN
+F 1 "TPH2R608NH" H 1856 3455 50  0000 L CNN
+F 2 "gesc:TRANS_TPHR8504PL-3PIN" H 1650 3500 50  0001 C CIN
+F 3 "" H 1650 3500 50  0001 L CNN
+F 4 "TPH2R608NH" H 2300 4500 236 0001 C CNN "Partnumber"
+F 5 "C146377" H 1950 4200 236 0001 C CNN "LCSC"
+	1    1650 3500
+	1    0    0    -1
+$EndComp
+$Comp
+L gesc:TPH2R608NH Q6
+U 1 1 604B5682
+P 1650 4150
+F 0 "Q6" H 1856 4196 50  0000 L CNN
+F 1 "TPH2R608NH" H 1856 4105 50  0000 L CNN
+F 2 "gesc:TRANS_TPHR8504PL-3PIN" H 1650 4150 50  0001 C CIN
+F 3 "" H 1650 4150 50  0001 L CNN
+F 4 "TPH2R608NH" H 2300 5150 236 0001 C CNN "Partnumber"
+F 5 "C146377" H 1950 4850 236 0001 C CNN "LCSC"
+	1    1650 4150
+	1    0    0    -1
+$EndComp
+$Comp
+L gesc:TPH2R608NH Q1
+U 1 1 604BC43D
+P 1600 5950
+F 0 "Q1" H 1806 5996 50  0000 L CNN
+F 1 "TPH2R608NH" H 1806 5905 50  0000 L CNN
+F 2 "gesc:TRANS_TPHR8504PL-3PIN" H 1600 5950 50  0001 C CIN
+F 3 "" H 1600 5950 50  0001 L CNN
+F 4 "TPH2R608NH" H 2250 6950 236 0001 C CNN "Partnumber"
+F 5 "C146377" H 1900 6650 236 0001 C CNN "LCSC"
+	1    1600 5950
+	1    0    0    -1
+$EndComp
+$Comp
+L gesc:TPH2R608NH Q2
+U 1 1 604BE734
+P 1600 6600
+F 0 "Q2" H 1806 6646 50  0000 L CNN
+F 1 "TPH2R608NH" H 1806 6555 50  0000 L CNN
+F 2 "gesc:TRANS_TPHR8504PL-3PIN" H 1600 6600 50  0001 C CIN
+F 3 "" H 1600 6600 50  0001 L CNN
+F 4 "TPH2R608NH" H 2250 7600 236 0001 C CNN "Partnumber"
+F 5 "C146377" H 1900 7300 236 0001 C CNN "LCSC"
+	1    1600 6600
+	1    0    0    -1
+$EndComp
 $EndSCHEMATC
