File: gesc_nrf.sch (KiCad schematic (older format))
At the start: 5 parts, among them J14 Conn_01x03, U16 EYSGJNZWY

Commit message: save
Parts:
- U16: footprint gsvesc:BLE_EYSGJNZWY -> gesc:BLE_EYSGJNZWY; symbol gsvesc:EYSGJNZWY -> gesc:EYSGJNZWY
Changed lines of the file:
@@
 encoding utf-8
 Sheet 2 5
-Title "GSESC - DC Motor Controler"
-Date "2018-11-11"
-Rev "4.0"
+Title "GESC - DC Motor Controler"
+Date "2020-04-09"
+Rev "6.0"
 Comp ""
 Comment1 ""
@@
 NRF_RX
 $Comp
-L gsvesc:EYSGJNZWY U16
+L gesc:EYSGJNZWY U16
 U 1 1 5E9F870E
 P 5100 4550
 F 0 "U16" H 5100 5617 50  0000 C CNN
 F 1 "EYSGJNZWY" H 5100 5526 50  0000 C CNN
-F 2 "gsvesc:BLE_EYSGJNZWY" H 5100 4550 50  0001 L BNN
+F 2 "gesc:BLE_EYSGJNZWY" H 5100 4550 50  0001 L BNN
 F 3 "Manufacturer Recommendation" H 5100 4550 50  0001 L BNN
 F 4 "1.3" H 5100 4550 50  0001 L BNN "Field4"

Commit message: save
Connections:
- net GND: now also J14.2 (Pin_2); no longer J14.1 (Pin_1)
- net at U16.16 (SWDIO): now also J14.3 (Pin_3); no longer J14.2 (Pin_2)
- net at U16.17 (SWDCLK): now also J14.1 (Pin_1); no longer J14.3 (Pin_3)
Other:
- moved on the sheet: J14
Changed lines of the file:
@@
 L Connector_Generic:Conn_01x03 J14
 U 1 1 5E9FAF5C
-P 3350 4350
-F 0 "J14" H 3270 4025 50  0000 C CNN
-F 1 "Conn_01x03" H 3270 4116 50  0000 C CNN
-F 2 "Connector_PinHeader_2.54mm:PinHeader_1x03_P2.54mm_Vertical" H 3350 4350 50  0001 C CNN
-F 3 "~" H 3350 4350 50  0001 C CNN
-	1    3350 4350
-	-1   0    0    1
+P 3050 4350
+F 0 "J14" H 3200 4350 50  0000 C CNN
+F 1 "Conn_01x03" H 3350 4450 50  0000 C CNN
+F 2 "Connector_PinHeader_2.54mm:PinHeader_1x03_P2.54mm_Vertical" H 3050 4350 50  0001 C CNN
+F 3 "~" H 3050 4350 50  0001 C CNN
+	1    3050 4350
+	-1   0    0    -1
 $EndComp
 Wire Wire Line
 	4000 4350 3550 4350
-Wire Wire Line
-	3550 4250 4000 4250
 $Comp
 L power:GND #PWR0158
 U 1 1 5E9FB3BA
-P 3550 4450
-F 0 "#PWR0158" H 3550 4200 50  0001 C CNN
-F 1 "GND" H 3650 4350 50  0000 C CNN
-F 2 "" H 3550 4450 50  0001 C CNN
-F 3 "" H 3550 4450 50  0001 C CNN
-	1    3550 4450
-	1    0    0    -1
+P 3250 4350
+F 0 "#PWR0158" H 3250 4100 50  0001 C CNN
+F 1 "GND" V 3250 4150 50  0000 C CNN
+F 2 "" H 3250 4350 50  0001 C CNN
+F 3 "" H 3250 4350 50  0001 C CNN
+	1    3250 4350
+	0    -1   -1   0
 $EndComp
+Wire Wire Line
+	3250 4250 4000 4250
+Wire Wire Line
+	3550 4350 3550 4450
+Wire Wire Line
+	3550 4450 3250 4450
 $EndSCHEMATC

Commit message: save
Parts:
- added TP1: Antenna, TestPoint:TestPoint_Pad_D2.0mm, symbol Connector:TestPoint
- added U18: RFM95W-868S2, gesc:XCVR_RFM95W-868S2, symbol RF_Module:RFM95W-868S2
Connections:
- net GND: now also U18.1 (GND), U18.10 (GND), U18.8 (GND)
- net VCC: now also U18.13 (3.3V)
- net NRF_RX renamed NRF_RX_MISO
- net NRF_RX_MISO: now also U18.2 (MISO)
- net NRF_TX renamed NRF_TX_SCK
- net NRF_TX_SCK: now also U18.4 (SCK)
- new net: TP1.1, U18.9 (ANT)
- new net DIO0: U18.14 (DIO0)
- new net MOSI: U18.3 (MOSI)
- new net NSS: U18.5 (NSS)
- new net RESET: U18.6 (RESET)
Changed lines of the file:
@@
 	4000 4650 3350 4650
 Text HLabel 3350 4650 0    50   Input ~ 0
-NRF_TX
+NRF_TX_SCK
 Text HLabel 3350 4750 0    50   Input ~ 0
-NRF_RX
+NRF_RX_MISO
 $Comp
 L gesc:EYSGJNZWY U16
@@
 Wire Wire Line
 	3550 4450 3250 4450
+$Comp
+L RF_Module:RFM95W-868S2 U18
+U 1 1 60528613
+P 4850 2450
+F 0 "U18" H 4250 3050 50  0000 C CNN
+F 1 "RFM95W-868S2" H 4450 2950 50  0000 C CNN
+F 2 "gesc:XCVR_RFM95W-868S2" H 1550 4100 50  0001 C CNN
+F 3 "https://www.hoperf.com/data/upload/portal/20181127/5bfcbea20e9ef.pdf" H 1550 4100 50  0001 C CNN
+	1    4850 2450
+	1    0    0    -1
+$EndComp
+Wire Wire Line
+	4350 2350 3600 2350
+Wire Wire Line
+	4350 2150 3600 2150
+Text HLabel 3600 2150 0    50   Input ~ 0
+NRF_TX_SCK
+Text HLabel 3600 2350 0    50   Input ~ 0
+NRF_RX_MISO
+Text HLabel 3600 2250 0    50   Input ~ 0
+MOSI
+Text HLabel 3600 2450 0    50   Input ~ 0
+NSS
+Text HLabel 3600 2650 0    50   Input ~ 0
+RESET
+Text HLabel 5650 2850 2    50   Input ~ 0
+DIO0
+Wire Wire Line
+	3600 2450 4350 2450
+Wire Wire Line
+	3600 2650 4350 2650
+Wire Wire Line
+	5350 2850 5650 2850
+$Comp
+L power:VCC #PWR0150
+U 1 1 6056EE55
+P 4850 1800
+F 0 "#PWR0150" H 4850 1650 50  0001 C CNN
+F 1 "VCC" V 4867 1928 50  0000 L CNN
+F 2 "" H 4850 1800 50  0001 C CNN
+F 3 "" H 4850 1800 50  0001 C CNN
+	1    4850 1800
+	1    0    0    -1
+$EndComp
+Wire Wire Line
+	4850 1800 4850 1950
+Wire Wire Line
+	4750 3150 4850 3150
+Wire Wire Line
+	4950 3150 4950 3050
+Wire Wire Line
+	4750 3150 4750 3050
+Wire Wire Line
+	4850 3050 4850 3150
+Connection ~ 4850 3150
+Wire Wire Line
+	4850 3150 4950 3150
+$Comp
+L power:GND #PWR0160
+U 1 1 60571C46
+P 4850 3150
+F 0 "#PWR0160" H 4850 2900 50  0001 C CNN
+F 1 "GND" H 4855 2977 50  0000 C CNN
+F 2 "" H 4850 3150 50  0001 C CNN
+F 3 "" H 4850 3150 50  0001 C CNN
+	1    4850 3150
+	1    0    0    -1
+$EndComp
+Wire Wire Line
+	3600 2250 4350 2250
+$Comp
+L Connector:TestPoint TP1
+U 1 1 605571D3
+P 5800 2150
+F 0 "TP1" H 5858 2268 50  0000 L CNN
+F 1 "Antenna" H 5858 2177 50  0000 L CNN
+F 2 "TestPoint:TestPoint_Pad_D2.0mm" H 6000 2150 50  0001 C CNN
+F 3 "~" H 6000 2150 50  0001 C CNN
+	1    5800 2150
+	1    0    0    -1
+$EndComp
+Wire Wire Line
+	5800 2150 5350 2150
 $EndSCHEMATC

Commit message: save
Connections:
- net NRF_RX_MISO: no longer U18.2 (MISO)
- net NRF_TX_SCK: no longer U18.4 (SCK)
- new net MISO: U18.2 (MISO)
- new net SCK: U18.4 (SCK)
Changed lines of the file:
@@
 	4350 2150 3600 2150
 Text HLabel 3600 2150 0    50   Input ~ 0
-NRF_TX_SCK
+SCK
 Text HLabel 3600 2350 0    50   Input ~ 0
-NRF_RX_MISO
+MISO
 Text HLabel 3600 2250 0    50   Input ~ 0
 MOSI
