File: gesc_uc.sch (KiCad schematic (older format))
At the start: 13 parts, among them U1 STM32F405RGTx, Y1 X50328MSB2GI

Commit message: - remove solder-mask from bottom layer
Parts:
- U1: LCSC (none) -> C15742
- Y1: LCSC (none) -> C115962
Changed lines of the file:
@@
 F 2 "Crystal:Crystal_SMD_5032-2Pin_5.0x3.2mm" H 1900 3900 50  0001 C CNN
 F 3 "~" H 1900 3900 50  0001 C CNN
+F 4 "C115962" V 1900 3900 50  0001 C CNN "LCSC"
 	1    1900 3900
 	0    1    1    0
@@
 F 2 "Package_QFP:LQFP-64_10x10mm_P0.5mm" H 3550 2500 50  0001 R CNN
 F 3 "http://www.st.com/st-web-ui/static/active/en/resource/technical/document/datasheet/DM00037051.pdf" H 4150 4200 50  0001 C CNN
+F 4 "C15742" H 4150 4200 50  0001 C CNN "LCSC"
 	1    4150 4200
 	1    0    0    -1

Commit message: save
Connections:
- net PA15 renamed SPI3_NSS
- net PC12 renamed SPI3_MOSI
- net P_UART_RX renamed P_UART_RX_MISO
- net P_UART_TX renamed P_UART_TX_SCK
Changed lines of the file:
@@
 $Descr A4 11693 8268
 encoding utf-8
-Sheet 3 5
+Sheet 5 5
 Title "GESC - DC Motor Controler"
 Date "2020-04-09"
@@
 Text HLabel 3200 4700 0    50   Input ~ 0
 TEMP_MOTOR
-Text HLabel 3200 4800 0    50   Input ~ 0
-PC5
 Text HLabel 3200 4900 0    50   Input ~ 0
 HALL_1
@@
 Connection ~ 2350 2600
 Text HLabel 5100 4100 2    50   Input ~ 0
-PA15
+SPI3_NSS
 Text HLabel 5100 4500 2    50   Input ~ 0
 PB2
@@
 Text HLabel 5100 4900 2    50   Input ~ 0
 PB6
-Text HLabel 3200 5300 0    50   Input ~ 0
-P_UART_TX
 Text HLabel 3200 5400 0    50   Input ~ 0
-P_UART_RX
+P_UART_RX_MISO
 Text HLabel 5100 5500 2    50   Input ~ 0
 PB12
@@
 	3200 5500 3450 5500
 Text HLabel 3200 5500 0    50   Input ~ 0
-PC12
+SPI3_MOSI
+Text HLabel 3200 4800 0    50   Input ~ 0
+PC5
+Text HLabel 3200 5300 0    50   Input ~ 0
+P_UART_TX_SCK
 $EndSCHEMATC

Commit message: save
Connections:
- net SPI3_MOSI renamed PC12
- net SPI3_NSS renamed PA15
Changed lines of the file:
@@
 Connection ~ 2350 2600
 Text HLabel 5100 4100 2    50   Input ~ 0
-SPI3_NSS
+PA15
 Text HLabel 5100 4500 2    50   Input ~ 0
 PB2
@@
 	3200 5500 3450 5500
 Text HLabel 3200 5500 0    50   Input ~ 0
-SPI3_MOSI
+PC12
 Text HLabel 3200 4800 0    50   Input ~ 0
 PC5
